File: Uni_stick/Uni_stick.kicad_pcb (KiCad board)
At the start: 2 copper layers, 62.5 x 95.8 mm, 59 parts, among them IC1 MPX5050DP, IC2 MPX5050DP, IC3 MAX20050ATC_V+, J1 Conn_01x04, J2 Conn_01x04, J3 Conn_01x06, J4 Micro match 6x2, J5 Conn_01x04, J6 Conn_01x06, J7 Conn_01x04, J8 Conn_01x06

Commit message: UPDATE - finished
Signed-off-by: Jacek <matuszewski.kartech@gmail.com>
Parts:
- removed C25: 100n, Capacitor_SMD:C_1206_3216Metric
- removed C26: 100n, Capacitor_SMD:C_0603_1608Metric
- removed IC3: MAX20050ATC_V+, myFootprints:SON50P300X300X80-13N
- removed L2: L_Small, Inductor_SMD:L_1206_3216Metric
- removed R13: 0,133R, Resistor_SMD:R_1206_3216Metric
- removed R16: R_Small, Resistor_SMD:R_0603_1608Metric
- removed RV1: R_POT, moje:3314J-1
- J1: footprint Connector_Phoenix_MC:PhoenixContact_MCV_1,5_4-G-3.5_1x04_P3.50mm_Vertical -> Connector_Phoenix_MC:PhoenixContact_MCV_1,5_2-G-3.5_1x02_P3.50mm_Vertical
- J4: footprint Biblioteki:CONN-TE-MICROMATCH-6X2-SMD_CORRECTED -> Connector_PinHeader_2.54mm:PinHeader_2x14_P2.54mm_Vertical; moved to B.Cu
- moved J4 70.4 mm to (81.5, 96.5), turned to 180 degrees
- moved C3 54.1 mm to (109.6, 65.2)
- moved C2 53.7 mm to (109.6, 59.7)
- moved C28 53.2 mm to (112.5, 55.9)
- moved R5 51.5 mm to (116.7, 124.8)
- moved R6 51.5 mm to (116.7, 122.5)
- moved SS3 51.4 mm to (114.4, 113.3)
- moved JP7 51.2 mm to (113.1, 123.7)
- moved J3 51.1 mm to (116.8, 77.9)
- moved JP3 51.1 mm to (118.9, 73.7)
- moved J8 51.0 mm to (106.1, 127.9)
- moved JP2 51.0 mm to (121.4, 73.7)
- moved JP1 51.0 mm to (123.9, 73.7)
- moved JP8 50.9 mm to (110.6, 123.7)
- moved R1 50.8 mm to (127.7, 74.8)
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Connections:
- J1 pad 1: +24V -> GND
- J1 pad 2: GND -> +24V
- J4 pad 1: /OUT_EXT1 -> (no net)
- J4 pad 10: /ADC_EXT_SEN1 -> (no net)
- J4 pad 11: GND -> /ADC_EXT_SEN2
- J4 pad 12: /ADC_EXT_SEN2 -> /ADC_EXT_SEN1
- J4 pad 2: /OUT_EXT2 -> (no net)
- J4 pad 3: /OUT_EXT3 -> /OUT_EXT2
- J4 pad 4: /OUT_EXT4 -> /OUT_EXT1
- J4 pad 5: /OUT_EXT5 -> /OUT_EXT4
- J4 pad 6: /OUT_EXT6 -> /OUT_EXT3
- J4 pad 7: +3V3 -> /OUT_EXT6
- J4 pad 8: /LIGHT_ON -> /OUT_EXT5
- J4 pad 9: +5V -> (no net)
Routing:
- net +24V: track 128.1 -> 0.00 mm
- net /LIGHT_ON: track 68.1 -> 0.00 mm, vias 4 -> 0
- net /OUT_EXT2: track 20.8 -> 74.5 mm, vias 1 -> 3
- net +5V: track 124.3 -> 170.4 mm
- net /OUT_EXT1: track 29.9 -> 75.7 mm, vias 1 -> 3
- net /ADC_EXT_SEN1: track 80.7 -> 126.0 mm, vias 2 -> 5
- net /OUT_EXT4: track 27.6 -> 64.6 mm, vias 1 -> 3
- net /OUT_EXT3: track 32.2 -> 64.2 mm, vias 1 -> 3
- net Net-(J2-Pad4): track 37.1 -> 56.7 mm
- net Net-(J2-Pad3): track 33.0 -> 51.3 mm
- net Net-(J2-Pad2): track 29.0 -> 44.7 mm, vias 1 -> 2
- net Net-(IC3-Pad3): track 15.4 -> 0.00 mm
- net Net-(J2-Pad1): track 25.3 -> 39.9 mm, vias 1 -> 2
- net Net-(C25-Pad1): track 11.7 -> 0.00 mm
- net Net-(J5-Pad4): track 44.5 -> 56.1 mm, vias 1 -> 2
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- added copper zone on F.Cu, net +24V
Other:
- board size 62.5 x 95.8 mm -> 68.4 x 95.8 mm
- net class Default removed
- board text removed: "CAN"
