File: Analog_digital_io.kicad_sch (KiCad schematic)
At the start: 4 parts, among them IC3 74HC14D

Commit message: Fixes
Signed-off-by: Jarosław Karwik <jaroslaw.karwik@gmail.com>
Parts:
- IC3: TME (none) -> SN74HC14DR
- RN6, RN7: TME (none) -> DR1206-100R-4/8
Changed lines of the file:
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@@
   (junction (at 125.095 60.96) (diameter 1.016) (color 0 0 0 0))
   (no_connect (at 130.175 77.47))
-  (no_connect (at 140.335 138.43))
   (no_connect (at 130.175 138.43))
   (no_connect (at 140.335 77.47))
+  (no_connect (at 140.335 138.43))
   (wire (pts (xy 90.805 69.85) (xy 94.615 69.85))
     (stroke (width 0) (type solid) (color 0 0 0 0))
@@
       (effects (font (size 1.524 1.524)))
     )
+    (property "TME" "SN74HC14DR" (id 4) (at 121.285 52.07 0)
+      (effects (font (size 1.27 1.27)) hide)
+    )
   )
   (symbol (lib_id "Uni_Printer-rescue:C-Device") (at 128.905 52.07 0) (unit 1)
@@
       (effects (font (size 1.27 1.27)) hide)
     )
+    (property "TME" "DR1206-100R-4/8" (id 4) (at 135.255 74.93 0)
+      (effects (font (size 1.27 1.27)) hide)
+    )
   )
   (symbol (lib_id "Uni_Printer-rescue:R_Pack04-Device") (at 135.255 135.89 270) (unit 1)
@@
       (effects (font (size 1.27 1.27)) hide)
     )
+    (property "TME" "DR1206-100R-4/8" (id 4) (at 135.255 135.89 0)
+      (effects (font (size 1.27 1.27)) hide)
+    )
   )
   (symbol (lib_id "Uni_Printer-rescue:74*14-step2cnc-Uni_Printer_v1-rescue") (at 104.775 69.85 0) (unit 6)
@@
       (effects (font (size 1.524 1.524)))
     )
+    (property "TME" "SN74HC14DR" (id 4) (at 104.775 69.85 0)
+      (effects (font (size 1.27 1.27)) hide)
+    )
   )
   (symbol (lib_id "Uni_Printer-rescue:74*14-step2cnc-Uni_Printer_v1-rescue") (at 104.775 81.28 0) (unit 5)
@@
       (effects (font (size 1.524 1.524)))
     )
+    (property "TME" "SN74HC14DR" (id 4) (at 104.775 81.28 0)
+      (effects (font (size 1.27 1.27)) hide)
+    )
   )
   (symbol (lib_id "Uni_Printer-rescue:74*14-step2cnc-Uni_Printer_v1-rescue") (at 104.775 92.71 0) (unit 4)
@@
       (effects (font (size 1.524 1.524)))
     )
+    (property "TME" "SN74HC14DR" (id 4) (at 104.775 92.71 0)
+      (effects (font (size 1.27 1.27)) hide)
+    )
   )
   (symbol (lib_id "Uni_Printer-rescue:74*14-step2cnc-Uni_Printer_v1-rescue") (at 104.775 106.68 0) (unit 3)
@@
       (effects (font (size 1.524 1.524)))
     )
+    (property "TME" "SN74HC14DR" (id 4) (at 104.775 106.68 0)
+      (effects (font (size 1.27 1.27)) hide)
+    )
   )
   (symbol (lib_id "Uni_Printer-rescue:74*14-step2cnc-Uni_Printer_v1-rescue") (at 104.775 120.65 0) (unit 2)
@@
       (effects (font (size 1.524 1.524)))
     )
+    (property "TME" "SN74HC14DR" (id 4) (at 104.775 120.65 0)
+      (effects (font (size 1.27 1.27)) hide)
+    )
   )
   (symbol (lib_id "Uni_Printer-rescue:74*14-step2cnc-Uni_Printer_v1-rescue") (at 104.775 135.89 0) (unit 1)
@@
       (effects (font (size 1.524 1.524)))
     )
-  )
+    (property "TME" "SN74HC14DR" (id 4) (at 104.775 135.89 0)
+      (effects (font (size 1.27 1.27)) hide)
+    )
+  )

Commit message: UPDATE - 3D and Jumper descriptions
Signed-off-by: Jacek <matuszewski.kartech@gmail.com>
Parts:
- C31: TME (none) -> C0603C104K3RAC
Changed lines of the file:
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@@
-(kicad_sch (version 20201015) (generator eeschema)
+(kicad_sch (version 20210126) (generator eeschema)
   (paper "A4")
   (title_block
@@
       (effects (font (size 1.27 1.27)) hide)
     )
+    (pin "1")
   )
   (symbol (lib_id "Uni_Printer-rescue:GND-Sensor_tank_v1-rescue-Uni_General_v1-rescue-Uni_Printer_v1-rescue") (at 125.095 63.5 0) (unit 1)
@@
       (effects (font (size 1.27 1.27)) hide)
     )
+    (pin "1")
   )
   (symbol (lib_id "Uni_Printer-rescue:74*14-step2cnc-Uni_Printer_v1-rescue") (at 121.285 52.07 0) (unit 7)
@@
       (effects (font (size 1.27 1.27)) hide)
     )
+    (pin "14")
+    (pin "7")
   )
   (symbol (lib_id "Uni_Printer-rescue:C-Device") (at 128.905 52.07 0) (unit 1)
@@
       (effects (font (size 1.27 1.27)) hide)
     )
+    (property "TME" "C0603C104K3RAC" (id 4) (at 128.905 52.07 0)
+      (effects (font (size 1.27 1.27)) hide)
+    )
+    (pin "1")
+    (pin "2")
   )
   (symbol (lib_id "Uni_Printer-rescue:R_Pack04-Device") (at 135.255 74.93 270) (unit 1)
@@
       (effects (font (size 1.27 1.27)) hide)
     )
+    (pin "1")
+    (pin "2")
+    (pin "3")
+    (pin "4")
+    (pin "5")
+    (pin "6")
+    (pin "7")
+    (pin "8")
   )
   (symbol (lib_id "Uni_Printer-rescue:R_Pack04-Device") (at 135.255 135.89 270) (unit 1)
@@
       (effects (font (size 1.27 1.27)) hide)
     )
+    (pin "1")
+    (pin "2")
+    (pin "3")
+    (pin "4")
+    (pin "5")
+    (pin "6")
+    (pin "7")
+    (pin "8")
   )
   (symbol (lib_id "Uni_Printer-rescue:74*14-step2cnc-Uni_Printer_v1-rescue") (at 104.775 69.85 0) (unit 6)
@@
       (effects (font (size 1.27 1.27)) hide)
     )
+    (pin "5")
+    (pin "6")
   )
   (symbol (lib_id "Uni_Printer-rescue:74*14-step2cnc-Uni_Printer_v1-rescue") (at 104.775 81.28 0) (unit 5)
@@
       (effects (font (size 1.27 1.27)) hide)
     )
+    (pin "3")
+    (pin "4")
   )
   (symbol (lib_id "Uni_Printer-rescue:74*14-step2cnc-Uni_Printer_v1-rescue") (at 104.775 92.71 0) (unit 4)
@@
       (effects (font (size 1.27 1.27)) hide)
     )
+    (pin "1")
+    (pin "2")
   )
   (symbol (lib_id "Uni_Printer-rescue:74*14-step2cnc-Uni_Printer_v1-rescue") (at 104.775 106.68 0) (unit 3)
@@
       (effects (font (size 1.27 1.27)) hide)
     )
+    (pin "8")
+    (pin "9")
   )
   (symbol (lib_id "Uni_Printer-rescue:74*14-step2cnc-Uni_Printer_v1-rescue") (at 104.775 120.65 0) (unit 2)
@@
       (effects (font (size 1.27 1.27)) hide)
     )
+    (pin "10")
+    (pin "11")
   )
   (symbol (lib_id "Uni_Printer-rescue:74*14-step2cnc-Uni_Printer_v1-rescue") (at 104.775 135.89 0) (unit 1)
@@
       (effects (font (size 1.27 1.27)) hide)
     )
+    (pin "12")
+    (pin "13")
   )
 )
