File: Encoder.kicad_sch (KiCad schematic)
At the start: 12 parts, among them U5 ST1480ACDR, U6 ST1480ACDR, U7 ST1480ACDR, U8 ST1480ACDR

Commit message: Fixes
Signed-off-by: Jarosław Karwik <jaroslaw.karwik@gmail.com>
Parts:
- C27, C28: TME C0603C104K3RAC -> (none)
- C30, R22, R23, R24, R25: TME WF06P-120R-5% -> (none)
- U5, U6, U7, U8: Category (none) -> Driver
Changed lines of the file:
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@@
   (junction (at 200.66 68.58) (diameter 1.016) (color 0 0 0 0))
   (junction (at 200.66 81.28) (diameter 1.016) (color 0 0 0 0))
-  (no_connect (at 172.72 123.19))
   (no_connect (at 93.98 80.01))
   (no_connect (at 93.98 124.46))
   (no_connect (at 172.72 78.74))
+  (no_connect (at 172.72 123.19))
   (wire (pts (xy 82.55 115.57) (xy 93.98 115.57))
     (stroke (width 0) (type solid) (color 0 0 0 0))
@@
       (effects (font (size 1.27 1.27)) hide)
     )
-    (property "TME" "WF06P-120R-5% " (id 4) (at 120.65 120.65 0)
+    (property "TME" "" (id 4) (at 120.65 120.65 0)
       (effects (font (size 1.27 1.27)) hide)
     )
@@
       (effects (font (size 1.27 1.27)) hide)
     )
-    (property "TME" "WF06P-120R-5% " (id 4) (at 121.92 76.2 0)
+    (property "TME" "" (id 4) (at 121.92 76.2 0)
       (effects (font (size 1.27 1.27)) hide)
     )
@@
       (effects (font (size 1.27 1.27)) hide)
     )
-    (property "TME" "WF06P-120R-5% " (id 4) (at 199.39 119.38 0)
+    (property "TME" "" (id 4) (at 199.39 119.38 0)
       (effects (font (size 1.27 1.27)) hide)
     )
@@
       (effects (font (size 1.27 1.27)) hide)
     )
-    (property "TME" "WF06P-120R-5% " (id 4) (at 200.66 74.93 0)
+    (property "TME" "" (id 4) (at 200.66 74.93 0)
       (effects (font (size 1.27 1.27)) hide)
     )
@@
       (effects (font (size 1.27 1.27)) hide)
     )
-    (property "TME" "C0603C104K3RAC" (id 4) (at 114.3 58.42 0)
+    (property "TME" "" (id 4) (at 114.3 58.42 0)
       (effects (font (size 1.27 1.27)) hide)
     )
@@
       (effects (font (size 1.27 1.27)) hide)
     )
-    (property "TME" "C0603C104K3RAC" (id 4) (at 114.3 102.87 0)
+    (property "TME" "" (id 4) (at 114.3 102.87 0)
       (effects (font (size 1.27 1.27)) hide)
     )
@@
       (effects (font (size 1.27 1.27)) hide)
     )
-    (property "TME" "WF06P-120R-5% " (id 4) (at 193.04 101.6 0)
+    (property "TME" "" (id 4) (at 193.04 101.6 0)
       (effects (font (size 1.27 1.27)) hide)
     )
@@
       (effects (font (size 1.27 1.27)) hide)
     )
+    (property "Category" "Driver" (id 4) (at 104.14 73.66 0)
+      (effects (font (size 1.27 1.27)) hide)
+    )
   )
   (symbol (lib_id "Uni_Printer-rescue:ST1480ACDR-Sensor_tank_v1-rescue-Uni_General_v1-rescue-Uni_Printer_v1-rescue") (at 104.14 118.11 0) (unit 1)
@@
       (effects (font (size 1.27 1.27)) hide)
     )
+    (property "Category" "Driver" (id 4) (at 104.14 118.11 0)
+      (effects (font (size 1.27 1.27)) hide)
+    )
   )
   (symbol (lib_id "Uni_Printer-rescue:ST1480ACDR-Sensor_tank_v1-rescue-Uni_General_v1-rescue-Uni_Printer_v1-rescue") (at 182.88 72.39 0) (unit 1)
@@
       (effects (font (size 1.27 1.27)) hide)
     )
+    (property "Category" "Driver" (id 4) (at 182.88 72.39 0)
+      (effects (font (size 1.27 1.27)) hide)
+    )
   )
   (symbol (lib_id "Uni_Printer-rescue:ST1480ACDR-Sensor_tank_v1-rescue-Uni_General_v1-rescue-Uni_Printer_v1-rescue") (at 182.88 116.84 0) (unit 1)
@@
       (effects (font (size 1.27 1.27)) hide)
     )
+    (property "Category" "Driver" (id 4) (at 182.88 116.84 0)
+      (effects (font (size 1.27 1.27)) hide)
+    )

Commit message: UPDATE - 3D and Jumper descriptions
Signed-off-by: Jacek <matuszewski.kartech@gmail.com>
Parts:
- C27, C28, C29, C30: TME (none) -> C0603C104K3RAC
- R22, R23, R24, R25: TME (none) -> WF06P-120R-5%
Changed lines of the file:
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@@
-(kicad_sch (version 20201015) (generator eeschema)
+(kicad_sch (version 20210126) (generator eeschema)
   (paper "A4")
   (title_block
@@
       (effects (font (size 1.27 1.27)) hide)
     )
+    (pin "1")
   )
   (symbol (lib_id "power:+3V3") (at 104.14 105.41 0) (unit 1)
@@
       (effects (font (size 1.27 1.27)) hide)
     )
+    (pin "1")
   )
   (symbol (lib_id "power:+3V3") (at 114.3 53.34 0) (unit 1)
@@
       (effects (font (size 1.27 1.27)) hide)
     )
+    (pin "1")
   )
   (symbol (lib_id "power:+3V3") (at 114.3 97.79 0) (unit 1)
@@
       (effects (font (size 1.27 1.27)) hide)
     )
+    (pin "1")
   )
   (symbol (lib_id "power:+3V3") (at 182.88 59.69 0) (unit 1)
@@
       (effects (font (size 1.27 1.27)) hide)
     )
+    (pin "1")
   )
   (symbol (lib_id "power:+3V3") (at 182.88 104.14 0) (unit 1)
@@
       (effects (font (size 1.27 1.27)) hide)
     )
+    (pin "1")
   )
   (symbol (lib_id "power:+3V3") (at 193.04 52.07 0) (unit 1)
@@
       (effects (font (size 1.27 1.27)) hide)
     )
+    (pin "1")
   )
   (symbol (lib_id "power:+3V3") (at 193.04 96.52 0) (unit 1)
@@
       (effects (font (size 1.27 1.27)) hide)
     )
+    (pin "1")
   )
   (symbol (lib_id "Uni_Printer-rescue:GND-power") (at 91.44 87.63 0) (unit 1)
@@
       (effects (font (size 1.27 1.27)) hide)
     )
+    (pin "1")
   )
   (symbol (lib_id "Uni_Printer-rescue:GND-power") (at 91.44 132.08 0) (unit 1)
@@
       (effects (font (size 1.27 1.27)) hide)
     )
+    (pin "1")
   )
   (symbol (lib_id "Uni_Printer-rescue:GND-power") (at 104.14 87.63 0) (unit 1)
@@
       (effects (font (size 1.27 1.27)) hide)
     )
+    (pin "1")
   )
   (symbol (lib_id "Uni_Printer-rescue:GND-power") (at 104.14 132.08 0) (unit 1)
@@
       (effects (font (size 1.27 1.27)) hide)
     )
+    (pin "1")
   )
   (symbol (lib_id "Uni_Printer-rescue:GND-power") (at 114.3 63.5 0) (unit 1)
@@
       (effects (font (size 1.27 1.27)) hide)
     )
+    (pin "1")
   )
   (symbol (lib_id "Uni_Printer-rescue:GND-power") (at 114.3 107.95 0) (unit 1)
@@
       (effects (font (size 1.27 1.27)) hide)
     )
+    (pin "1")
   )
   (symbol (lib_id "Uni_Printer-rescue:GND-power") (at 170.18 86.36 0) (unit 1)
@@
       (effects (font (size 1.27 1.27)) hide)
     )
+    (pin "1")
   )
   (symbol (lib_id "Uni_Printer-rescue:GND-power") (at 170.18 130.81 0) (unit 1)
@@
       (effects (font (size 1.27 1.27)) hide)
     )
+    (pin "1")
   )
   (symbol (lib_id "Uni_Printer-rescue:GND-power") (at 182.88 86.36 0) (unit 1)
@@
       (effects (font (size 1.27 1.27)) hide)
     )
+    (pin "1")
   )
   (symbol (lib_id "Uni_Printer-rescue:GND-power") (at 182.88 130.81 0) (unit 1)
@@
       (effects (font (size 1.27 1.27)) hide)
     )
+    (pin "1")
   )
   (symbol (lib_id "Uni_Printer-rescue:GND-power") (at 193.04 62.23 0) (unit 1)
@@
       (effects (font (size 1.27 1.27)) hide)
     )
+    (pin "1")
   )
   (symbol (lib_id "Uni_Printer-rescue:GND-power") (at 193.04 106.68 0) (unit 1)
@@
       (effects (font (size 1.27 1.27)) hide)
     )
+    (pin "1")
   )
   (symbol (lib_id "Uni_Printer-rescue:R-Device") (at 120.65 120.65 0) (unit 1)
@@
       (effects (font (size 1.27 1.27)) hide)
     )
-    (property "TME" "" (id 4) (at 120.65 120.65 0)
-      (effects (font (size 1.27 1.27)) hide)
-    )
+    (property "TME" "WF06P-120R-5%" (id 4) (at 120.65 120.65 0)
+      (effects (font (size 1.27 1.27)) hide)
+    )
+    (pin "1")
+    (pin "2")
   )
   (symbol (lib_id "Uni_Printer-rescue:R-Device") (at 121.92 76.2 0) (unit 1)
@@
       (effects (font (size 1.27 1.27)) hide)
     )
-    (property "TME" "" (id 4) (at 121.92 76.2 0)
-      (effects (font (size 1.27 1.27)) hide)
-    )
+    (property "TME" "WF06P-120R-5%" (id 4) (at 121.92 76.2 0)
+      (effects (font (size 1.27 1.27)) hide)
+    )
+    (pin "1")
+    (pin "2")
   )
   (symbol (lib_id "Uni_Printer-rescue:R-Device") (at 199.39 119.38 0) (unit 1)
@@
       (effects (font (size 1.27 1.27)) hide)
     )
-    (property "TME" "" (id 4) (at 199.39 119.38 0)
-      (effects (font (size 1.27 1.27)) hide)
-    )
+    (property "TME" "WF06P-120R-5%" (id 4) (at 199.39 119.38 0)
+      (effects (font (size 1.27 1.27)) hide)
+    )
+    (pin "1")
+    (pin "2")
   )
   (symbol (lib_id "Uni_Printer-rescue:R-Device") (at 200.66 74.93 0) (unit 1)
@@
       (effects (font (size 1.27 1.27)) hide)
     )
-    (property "TME" "" (id 4) (at 200.66 74.93 0)
-      (effects (font (size 1.27 1.27)) hide)
-    )
+    (property "TME" "WF06P-120R-5%" (id 4) (at 200.66 74.93 0)
+      (effects (font (size 1.27 1.27)) hide)
+    )
+    (pin "1")
+    (pin "2")
   )
   (symbol (lib_id "Uni_Printer-rescue:C_Small-Device") (at 114.3 58.42 0) (unit 1)
@@
       (effects (font (size 1.27 1.27)) hide)
     )
-    (property "TME" "" (id 4) (at 114.3 58.42 0)
-      (effects (font (size 1.27 1.27)) hide)
-    )
+    (property "TME" "C0603C104K3RAC" (id 4) (at 114.3 58.42 0)
+      (effects (font (size 1.27 1.27)) hide)
+    )
+    (pin "1")
+    (pin "2")
   )
   (symbol (lib_id "Uni_Printer-rescue:C_Small-Device") (at 114.3 102.87 0) (unit 1)
@@
       (effects (font (size 1.27 1.27)) hide)
     )
-    (property "TME" "" (id 4) (at 114.3 102.87 0)
-      (effects (font (size 1.27 1.27)) hide)
-    )
+    (property "TME" "C0603C104K3RAC" (id 4) (at 114.3 102.87 0)
+      (effects (font (size 1.27 1.27)) hide)
+    )
+    (pin "1")
+    (pin "2")
   )
   (symbol (lib_id "Uni_Printer-rescue:C_Small-Device") (at 193.04 57.15 0) (unit 1)
@@
       (effects (font (size 1.27 1.27)) hide)
     )
+    (property "TME" "C0603C104K3RAC" (id 4) (at 193.04 57.15 0)
+      (effects (font (size 1.27 1.27)) hide)
+    )
+    (pin "1")
+    (pin "2")
   )
   (symbol (lib_id "Uni_Printer-rescue:C_Small-Device") (at 193.04 101.6 0) (unit 1)
@@
       (effects (font (size 1.27 1.27)) hide)
     )
-    (property "TME" "" (id 4) (at 193.04 101.6 0)
-      (effects (font (size 1.27 1.27)) hide)
-    )
+    (property "TME" "C0603C104K3RAC" (id 4) (at 193.04 101.6 0)
+      (effects (font (size 1.27 1.27)) hide)
+    )
+    (pin "1")
+    (pin "2")
   )
   (symbol (lib_id "Uni_Printer-rescue:ST1480ACDR-Sensor_tank_v1-rescue-Uni_General_v1-rescue-Uni_Printer_v1-rescue") (at 104.14 73.66 0) (unit 1)
@@
       (effects (font (size 1.27 1.27)) hide)
     )
+    (pin "1")
+    (pin "2")
+    (pin "3")
+    (pin "4")
+    (pin "5")
+    (pin "6")
+    (pin "7")
+    (pin "8")
   )
   (symbol (lib_id "Uni_Printer-rescue:ST1480ACDR-Sensor_tank_v1-rescue-Uni_General_v1-rescue-Uni_Printer_v1-rescue") (at 104.14 118.11 0) (unit 1)
@@
       (effects (font (size 1.27 1.27)) hide)
     )
+    (pin "1")
+    (pin "2")
+    (pin "3")
+    (pin "4")
+    (pin "5")
+    (pin "6")
+    (pin "7")
+    (pin "8")
   )
   (symbol (lib_id "Uni_Printer-rescue:ST1480ACDR-Sensor_tank_v1-rescue-Uni_General_v1-rescue-Uni_Printer_v1-rescue") (at 182.88 72.39 0) (unit 1)
@@
       (effects (font (size 1.27 1.27)) hide)
     )
+    (pin "1")
+    (pin "2")
+    (pin "3")
+    (pin "4")
+    (pin "5")
+    (pin "6")
+    (pin "7")
+    (pin "8")
   )
   (symbol (lib_id "Uni_Printer-rescue:ST1480ACDR-Sensor_tank_v1-rescue-Uni_General_v1-rescue-Uni_Printer_v1-rescue") (at 182.88 116.84 0) (unit 1)
@@
       (effects (font (size 1.27 1.27)) hide)
     )
+    (pin "1")
+    (pin "2")
+    (pin "3")
+    (pin "4")
+    (pin "5")
+    (pin "6")
+    (pin "7")
+    (pin "8")
   )
 )
