File: Outputs.kicad_sch (KiCad schematic)
At the start: 8 parts, among them IC10 ITS4141NHUMA1, IC11 ITS4141NHUMA1, IC6 ITS4141NHUMA1, IC7 ITS4141NHUMA1, IC8 ITS4141NHUMA1, IC9 ITS4141NHUMA1

Commit message: Fixes
Signed-off-by: Jarosław Karwik <jaroslaw.karwik@gmail.com>
Parts:
- IC10, IC11, IC6, IC7, IC8, IC9: TME (none) -> TS4141N
- RN12, RN13: value 15k -> 10k; TME (none) -> DR1206-10K-4/8
Changed lines of the file:
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@@
   (junction (at 151.13 36.83) (diameter 1.016) (color 0 0 0 0))
   (junction (at 151.13 39.37) (diameter 1.016) (color 0 0 0 0))
+  (no_connect (at 140.335 59.69))
   (no_connect (at 140.335 62.23))
-  (no_connect (at 140.335 59.69))
   (wire (pts (xy 34.925 98.425) (xy 24.765 98.425))
     (stroke (width 0) (type solid) (color 0 0 0 0))
@@
     (in_bom yes) (on_board yes)
     (property "Reference" "RN12" (id 0) (at 145.415 49.0982 90))
-    (property "Value" "15k" (id 1) (at 145.415 51.41 90))
+    (property "Value" "10k" (id 1) (at 145.415 51.41 90))
     (property "Footprint" "moje:R_Array_Convex_4x0603" (id 2) (at 145.415 66.675 90)
       (effects (font (size 1.27 1.27)) hide)
@@
       (effects (font (size 1.27 1.27)) hide)
     )
+    (property "TME" "DR1206-10K-4/8" (id 4) (at 145.415 59.69 0)
+      (effects (font (size 1.27 1.27)) hide)
+    )
   )
   (symbol (lib_id "Uni_Printer-rescue:R_Pack04-Device") (at 146.05 36.83 270) (unit 1)
     (in_bom yes) (on_board yes)
     (property "Reference" "RN13" (id 0) (at 146.05 26.2382 90))
-    (property "Value" "15k" (id 1) (at 146.05 28.55 90))
+    (property "Value" "10k" (id 1) (at 146.05 28.55 90))
     (property "Footprint" "moje:R_Array_Convex_4x0603" (id 2) (at 146.05 43.815 90)
       (effects (font (size 1.27 1.27)) hide)
     )
     (property "Datasheet" "~" (id 3) (at 146.05 36.83 0)
+      (effects (font (size 1.27 1.27)) hide)
+    )
+    (property "TME" "DR1206-10K-4/8" (id 4) (at 146.05 36.83 0)
       (effects (font (size 1.27 1.27)) hide)
     )
@@
       (effects (font (size 1.27 1.27)) (justify left) hide)
     )
+    (property "TME" "TS4141N" (id 4) (at 34.925 98.425 0)
+      (effects (font (size 1.27 1.27)) hide)
+    )
   )
   (symbol (lib_id "ITS4141NHUMA1:ITS4141NHUMA1") (at 34.925 115.57 0) (unit 1)
@@
       (effects (font (size 1.27 1.27)) (justify left) hide)
     )
+    (property "TME" "TS4141N" (id 4) (at 34.925 115.57 0)
+      (effects (font (size 1.27 1.27)) hide)
+    )
   )
   (symbol (lib_id "ITS4141NHUMA1:ITS4141NHUMA1") (at 35.56 29.845 0) (unit 1)
@@
       (effects (font (size 1.27 1.27)) (justify left) hide)
     )
+    (property "TME" "TS4141N" (id 4) (at 35.56 29.845 0)
+      (effects (font (size 1.27 1.27)) hide)
+    )
   )
   (symbol (lib_id "ITS4141NHUMA1:ITS4141NHUMA1") (at 35.56 47.625 0) (unit 1)
@@
       (effects (font (size 1.27 1.27)) (justify left) hide)
     )
+    (property "TME" "TS4141N" (id 4) (at 35.56 47.625 0)
+      (effects (font (size 1.27 1.27)) hide)
+    )
   )
   (symbol (lib_id "ITS4141NHUMA1:ITS4141NHUMA1") (at 35.56 64.135 0) (unit 1)
@@
       (effects (font (size 1.27 1.27)) (justify left) hide)
     )
+    (property "TME" "TS4141N" (id 4) (at 35.56 64.135 0)
+      (effects (font (size 1.27 1.27)) hide)
+    )
   )
   (symbol (lib_id "ITS4141NHUMA1:ITS4141NHUMA1") (at 35.56 81.28 0) (unit 1)
@@
       (effects (font (size 1.27 1.27)) (justify left) hide)
     )
-  )
+    (property "TME" "TS4141N" (id 4) (at 35.56 81.28 0)
+      (effects (font (size 1.27 1.27)) hide)
+    )
+  )
