File: Power_supply.kicad_sch (KiCad schematic)
At the start: 12 parts, among them IC1 MAX17503ATP+, IC4 TLV1117-33

Commit message: Fixes
Signed-off-by: Jarosław Karwik <jaroslaw.karwik@gmail.com>
Parts:
- C1: value 100nF -> 100n
- C40: TME (none) -> 1210B106K500CT
- C43: footprint Capacitor_SMD:C_1206_3216Metric -> Capacitor_SMD:C_1210_3225Metric; TME (none) -> CL32A226KAJNNNE
- C44: TME (none) -> 293D107X96R3D2TE3
- IC1: Digi (none) -> MAX17503ATP+-ND
Changed lines of the file:
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@@
   (junction (at 193.167 76.835) (diameter 1.016) (color 0 0 0 0))
   (junction (at 233.553 67.31) (diameter 1.016) (color 0 0 0 0))
+  (no_connect (at 137.795 118.745))
   (no_connect (at 142.875 118.745))
-  (no_connect (at 137.795 118.745))
+  (no_connect (at 147.955 118.745))
   (no_connect (at 160.655 103.505))
-  (no_connect (at 147.955 118.745))
   (wire (pts (xy 85.09 93.345) (xy 92.71 93.345))
     (stroke (width 0) (type solid) (color 0 0 0 0))
@@
       (effects (font (size 1.27 1.27)) hide)
     )
+    (property "TME" "1210B106K500CT" (id 4) (at 118.745 95.885 0)
+      (effects (font (size 1.27 1.27)) hide)
+    )
   )
   (symbol (lib_id "Device:C_Small") (at 140.335 67.31 90) (unit 1)
     (in_bom yes) (on_board yes)
     (property "Reference" "C1" (id 0) (at 140.335 64.77 90))
-    (property "Value" "100nF" (id 1) (at 140.335 62.23 90))
+    (property "Value" "100n" (id 1) (at 140.335 62.23 90))
     (property "Footprint" "Capacitor_SMD:C_0603_1608Metric" (id 2) (at 140.335 67.31 0)
       (effects (font (size 1.27 1.27)) hide)
@@
       (effects (font (size 1.27 1.27)) (justify left))
     )
-    (property "Footprint" "Capacitor_SMD:C_1206_3216Metric" (id 2) (at 181.991 70.231 0)
+    (property "Footprint" "Capacitor_SMD:C_1210_3225Metric" (id 2) (at 181.991 70.231 0)
       (effects (font (size 1.27 1.27)) hide)
     )
@@
       (effects (font (size 1.27 1.27)) hide)
     )
+    (property "TME" "CL32A226KAJNNNE" (id 4) (at 181.991 70.231 0)
+      (effects (font (size 1.27 1.27)) hide)
+    )
   )
   (symbol (lib_id "Device:C_Small") (at 233.553 71.12 0) (unit 1)
@@
     )
     (property "Datasheet" "~" (id 3) (at 233.553 71.12 0)
+      (effects (font (size 1.27 1.27)) hide)
+    )
+    (property "TME" "293D107X96R3D2TE3" (id 4) (at 233.553 71.12 0)
       (effects (font (size 1.27 1.27)) hide)
     )
@@
       (effects (font (size 1.27 1.27)) (justify left) hide)
     )
-  )
+    (property "Digi" "MAX17503ATP+-ND" (id 4) (at 125.095 93.345 0)
+      (effects (font (size 1.27 1.27)) hide)
+    )
+  )

Commit message: UPDATE - 3D and Jumper descriptions
Signed-off-by: Jacek <matuszewski.kartech@gmail.com>
Parts:
- C1: TME (none) -> C0603C104K3RAC
- C41: TME (none) -> CL10A225KP8NNNC
- C42: TME (none) -> 0603B562K500CT
- R52: TME (none) -> CQ0603-180K-1%
- R53: TME (none) -> WF06P-39K-5%
Changed lines of the file:
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@@
-(kicad_sch (version 20201015) (generator eeschema)
+(kicad_sch (version 20210126) (generator eeschema)
   (paper "A4")
   (title_block
@@
       (effects (font (size 1.27 1.27)) hide)
     )
+    (pin "1")
+    (pin "2")
   )
   (symbol (lib_id "power:+5V") (at 193.167 65.151 0) (unit 1)
@@
       (effects (font (size 1.27 1.27)) hide)
     )
+    (pin "1")
   )
   (symbol (lib_id "power:+3V3") (at 233.553 65.532 0) (unit 1)
@@
       (effects (font (size 1.27 1.27)) hide)
     )
+    (pin "1")
   )
   (symbol (lib_id "power:GND") (at 92.71 100.965 0) (unit 1)
@@
       (effects (font (size 1.27 1.27)) hide)
     )
+    (pin "1")
   )
   (symbol (lib_id "power:GND") (at 118.745 98.425 0) (unit 1)
@@
       (effects (font (size 1.27 1.27)) hide)
     )
+    (pin "1")
   )
   (symbol (lib_id "power:GND") (at 135.255 75.565 180) (unit 1)
@@
       (effects (font (size 1.27 1.27)) hide)
     )
+    (pin "1")
   )
   (symbol (lib_id "power:GND") (at 140.335 126.111 0) (unit 1)
@@
       (effects (font (size 1.27 1.27)) hide)
     )
+    (pin "1")
   )
   (symbol (lib_id "power:GND") (at 147.955 75.565 180) (unit 1)
@@
       (effects (font (size 1.27 1.27)) hide)
     )
+    (pin "1")
   )
   (symbol (lib_id "power:GND") (at 160.655 95.885 90) (unit 1)
@@
       (effects (font (size 1.27 1.27)) hide)
     )
+    (pin "1")
   )
   (symbol (lib_id "power:GND") (at 167.513 106.045 0) (unit 1)
@@
       (effects (font (size 1.27 1.27)) hide)
     )
+    (pin "1")
   )
   (symbol (lib_id "power:GND") (at 181.991 72.771 0) (unit 1)
@@
       (effects (font (size 1.27 1.27)) hide)
     )
+    (pin "1")
   )
   (symbol (lib_id "power:GND") (at 193.167 85.471 0) (unit 1)
@@
       (effects (font (size 1.27 1.27)) hide)
     )
+    (pin "1")
   )
   (symbol (lib_id "power:GND") (at 215.265 76.2 0) (unit 1)
@@
       (effects (font (size 1.27 1.27)) hide)
     )
+    (pin "1")
   )
   (symbol (lib_id "power:GND") (at 233.553 73.66 0) (unit 1)
@@
       (effects (font (size 1.27 1.27)) hide)
     )
+    (pin "1")
   )
   (symbol (lib_id "Device:R_Small") (at 193.167 71.501 0) (unit 1)
@@
       (effects (font (size 1.27 1.27)) hide)
     )
+    (property "TME" "CQ0603-180K-1%" (id 4) (at 193.167 71.501 0)
+      (effects (font (size 1.27 1.27)) hide)
+    )
+    (pin "1")
+    (pin "2")
   )
   (symbol (lib_id "Device:R_Small") (at 193.167 82.931 0) (unit 1)
@@
       (effects (font (size 1.27 1.27)) hide)
     )
+    (property "TME" "WF06P-39K-5%" (id 4) (at 193.167 82.931 0)
+      (effects (font (size 1.27 1.27)) hide)
+    )
+    (pin "1")
+    (pin "2")
   )
   (symbol (lib_id "Device:C_Small") (at 118.745 95.885 0) (unit 1)
@@
       (effects (font (size 1.27 1.27)) hide)
     )
+    (pin "1")
+    (pin "2")
   )
   (symbol (lib_id "Device:C_Small") (at 140.335 67.31 90) (unit 1)
@@
       (effects (font (size 1.27 1.27)) hide)
     )
+    (property "TME" "C0603C104K3RAC" (id 4) (at 140.335 67.31 0)
+      (effects (font (size 1.27 1.27)) hide)
+    )
+    (pin "1")
+    (pin "2")
   )
   (symbol (lib_id "Device:C_Small") (at 140.335 123.571 180) (unit 1)
@@
       (effects (font (size 1.27 1.27)) hide)
     )
+    (property "TME" "0603B562K500CT" (id 4) (at 140.335 123.571 0)
+      (effects (font (size 1.27 1.27)) hide)
+    )
+    (pin "1")
+    (pin "2")
   )
   (symbol (lib_id "Device:C_Small") (at 167.513 103.505 0) (unit 1)
@@
       (effects (font (size 1.27 1.27)) hide)
     )
+    (property "TME" "CL10A225KP8NNNC" (id 4) (at 167.513 103.505 0)
+      (effects (font (size 1.27 1.27)) hide)
+    )
+    (pin "1")
+    (pin "2")
   )
   (symbol (lib_id "Device:C_Small") (at 181.991 70.231 0) (unit 1)
@@
       (effects (font (size 1.27 1.27)) hide)
     )
+    (pin "1")
+    (pin "2")
   )
   (symbol (lib_id "Device:C_Small") (at 233.553 71.12 0) (unit 1)
@@
       (effects (font (size 1.27 1.27)) hide)
     )
+    (pin "1")
+    (pin "2")
   )
   (symbol (lib_id "Device:D_TVS") (at 92.71 97.155 90) (unit 1)
@@
       (effects (font (size 1.27 1.27)) hide)
     )
+    (pin "1")
+    (pin "2")
   )
   (symbol (lib_id "DriveAdd_Printer_v2-rescue:LM1117-step2cnc-Sensor_tank_v1-rescue-Uni_General_v1-rescue-Uni_Printer_v1-rescue-Uni_Printer-rescue") (at 215.265 67.31 0) (unit 1)
@@
       (effects (font (size 1.27 1.27)) hide)
     )
+    (pin "1")
+    (pin "2")
+    (pin "3")
   )
   (symbol (lib_id "MAX17503ATP+:MAX17503ATP+") (at 125.095 93.345 0) (unit 1)
@@
       (effects (font (size 1.27 1.27)) hide)
     )
+    (pin "1")
+    (pin "2")
+    (pin "3")
+    (pin "4")
+    (pin "5")
+    (pin "6")
+    (pin "7")
+    (pin "8")
+    (pin "9")
+    (pin "10")
+    (pin "15")
+    (pin "14")
+    (pin "13")
+    (pin "12")
+    (pin "11")
+    (pin "21")
+    (pin "20")
+    (pin "19")
+    (pin "18")
+    (pin "17")
+    (pin "16")
   )
 )
