File: RS485_CAN.kicad_sch (KiCad schematic)
At the start: 9 parts, among them U3 TLE9251VSJ, U9 ST1480ACDR

Commit message: Fixes
Signed-off-by: Jarosław Karwik <jaroslaw.karwik@gmail.com>
Parts:
- C2, C3: Category Capacitor -> (none)
- C32: TME C0603C104K3RAC -> (none)
- R39, R40: TME WF06P-120R-5% -> (none)
- U9: Category (none) -> Driver; TME SP3485EN-L -> SP3077EEN-L
Changed lines of the file:
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@@
       (effects (font (size 1.27 1.27)) hide)
     )
-    (property "TME" "WF06P-120R-5% " (id 4) (at 105.41 49.53 90)
+    (property "TME" "" (id 4) (at 105.41 49.53 90)
       (effects (font (size 1.27 1.27)) hide)
     )
@@
       (effects (font (size 1.27 1.27)) hide)
     )
-    (property "TME" "WF06P-120R-5% " (id 4) (at 105.41 96.52 90)
+    (property "TME" "" (id 4) (at 105.41 96.52 90)
       (effects (font (size 1.27 1.27)) hide)
     )
@@
       (effects (font (size 1.27 1.27)) hide)
     )
-    (property "TME" "C0603C104K3RAC" (id 4) (at 83.82 26.67 0)
+    (property "TME" "" (id 4) (at 83.82 26.67 0)
       (effects (font (size 1.27 1.27)) hide)
     )
@@
       (effects (font (size 1.27 1.27)) hide)
     )
-    (property "Category" "Capacitor" (id 4) (at 36.83 69.85 0)
+    (property "Category" "" (id 4) (at 36.83 69.85 0)
       (effects (font (size 1.524 1.524)) hide)
     )
@@
       (effects (font (size 1.27 1.27)) hide)
     )
-    (property "Category" "Capacitor" (id 4) (at 52.07 69.85 0)
+    (property "Category" "" (id 4) (at 52.07 69.85 0)
       (effects (font (size 1.524 1.524)) hide)
     )
@@
       (effects (font (size 1.27 1.27)) hide)
     )
-    (property "TME" "SP3485EN-L" (id 4) (at 78.74 36.83 0)
+    (property "TME" "SP3077EEN-L " (id 4) (at 78.74 36.83 0)
       (effects (font (size 1.27 1.27)) hide)
     )
+    (property "Category" "Driver" (id 4) (at 78.74 36.83 0)
+      (effects (font (size 1.27 1.27)) hide)
+    )

Commit message: UPDATE - 3D and Jumper descriptions
Signed-off-by: Jacek <matuszewski.kartech@gmail.com>
Parts:
- C2, C3, C32: TME (none) -> C0603C104K3RAC
- R39, R40: TME (none) -> WF06P-120R-5%
Changed lines of the file:
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@@
-(kicad_sch (version 20201015) (generator eeschema)
+(kicad_sch (version 20210126) (generator eeschema)
   (paper "A4")
   (title_block
@@
       (effects (font (size 1.27 1.27)) hide)
     )
+    (pin "1")
+    (pin "2")
   )
   (symbol (lib_id "Uni_Printer-rescue:Jumper_NO_Small-Device") (at 105.41 80.01 90) (unit 1)
@@
       (effects (font (size 1.27 1.27)) hide)
     )
+    (pin "1")
+    (pin "2")
   )
   (symbol (lib_id "power:+5V") (at 36.83 66.04 0) (unit 1)
@@
       (effects (font (size 1.27 1.27)) hide)
     )
+    (pin "1")
   )
   (symbol (lib_id "power:+3V3") (at 52.07 66.04 0) (unit 1)
@@
       (effects (font (size 1.27 1.27)) hide)
     )
+    (pin "1")
   )
   (symbol (lib_id "power:+3V3") (at 64.77 87.63 90) (unit 1)
@@
       (effects (font (size 1.27 1.27)) hide)
     )
+    (pin "1")
   )
   (symbol (lib_id "power:+5V") (at 77.47 72.39 0) (unit 1)
@@
       (effects (font (size 1.27 1.27)) hide)
     )
+    (pin "1")
   )
   (symbol (lib_id "power:+3V3") (at 78.74 24.13 0) (unit 1)
@@
       (effects (font (size 1.27 1.27)) hide)
     )
+    (pin "1")
   )
   (symbol (lib_id "mfc_base_lib:GND") (at 36.83 73.66 0) (unit 1)
@@
       (effects (font (size 1.27 1.27)) hide)
     )
+    (pin "1")
   )
   (symbol (lib_id "mfc_base_lib:GND") (at 52.07 73.66 0) (unit 1)
@@
       (effects (font (size 1.27 1.27)) hide)
     )
+    (pin "1")
   )
   (symbol (lib_id "mfc_base_lib:GND") (at 64.77 92.71 270) (unit 1)
@@
       (effects (font (size 1.27 1.27)) hide)
     )
+    (pin "1")
   )
   (symbol (lib_id "mfc_base_lib:GND") (at 77.47 107.95 0) (unit 1)
@@
       (effects (font (size 1.27 1.27)) hide)
     )
+    (pin "1")
   )
   (symbol (lib_id "Uni_Printer-rescue:GND-Sensor_tank_v1-rescue-Uni_General_v1-rescue-Uni_Printer_v1-rescue") (at 78.74 50.8 0) (unit 1)
@@
       (effects (font (size 1.27 1.27)) hide)
     )
+    (pin "1")
   )
   (symbol (lib_id "Uni_Printer-rescue:GND-Sensor_tank_v1-rescue-Uni_General_v1-rescue-Uni_Printer_v1-rescue") (at 88.9 29.21 0) (unit 1)
@@
       (effects (font (size 1.27 1.27)) hide)
     )
+    (pin "1")
   )
   (symbol (lib_id "Uni_Printer-rescue:R-Sensor_tank_v1-rescue-Uni_General_v1-rescue-Uni_Printer_v1-rescue") (at 105.41 49.53 0) (unit 1)
@@
       (effects (font (size 1.27 1.27)) hide)
     )
-    (property "TME" "" (id 4) (at 105.41 49.53 90)
-      (effects (font (size 1.27 1.27)) hide)
-    )
+    (property "TME" "WF06P-120R-5%" (id 4) (at 105.41 49.53 90)
+      (effects (font (size 1.27 1.27)) hide)
+    )
+    (pin "1")
+    (pin "2")
   )
   (symbol (lib_id "Uni_Printer-rescue:R-Sensor_tank_v1-rescue-Uni_General_v1-rescue-Uni_Printer_v1-rescue") (at 105.41 96.52 0) (unit 1)
@@
       (effects (font (size 1.27 1.27)) hide)
     )
-    (property "TME" "" (id 4) (at 105.41 96.52 90)
-      (effects (font (size 1.27 1.27)) hide)
-    )
+    (property "TME" "WF06P-120R-5%" (id 4) (at 105.41 96.52 90)
+      (effects (font (size 1.27 1.27)) hide)
+    )
+    (pin "1")
+    (pin "2")
   )
   (symbol (lib_id "Uni_Printer-rescue:C_Small-Sensor_tank_v1-rescue-Uni_General_v1-rescue-Uni_Printer_v1-rescue") (at 83.82 26.67 90) (unit 1)
@@
       (effects (font (size 1.27 1.27)) hide)
     )
-    (property "TME" "" (id 4) (at 83.82 26.67 0)
-      (effects (font (size 1.27 1.27)) hide)
-    )
+    (property "TME" "C0603C104K3RAC" (id 4) (at 83.82 26.67 0)
+      (effects (font (size 1.27 1.27)) hide)
+    )
+    (pin "1")
+    (pin "2")
   )
   (symbol (lib_id "mfc_base_lib:C") (at 36.83 69.85 0) (unit 1)
@@
       (effects (font (size 1.524 1.524)) hide)
     )
+    (property "TME" "C0603C104K3RAC" (id 4) (at 36.83 69.85 0)
+      (effects (font (size 1.27 1.27)) hide)
+    )
+    (pin "1")
+    (pin "2")
   )
   (symbol (lib_id "mfc_base_lib:C") (at 52.07 69.85 0) (unit 1)
@@
       (effects (font (size 1.524 1.524)) hide)
     )
+    (property "TME" "C0603C104K3RAC" (id 4) (at 52.07 69.85 0)
+      (effects (font (size 1.27 1.27)) hide)
+    )
+    (pin "1")
+    (pin "2")
   )
   (symbol (lib_id "Uni_Printer-rescue:ST1480ACDR-Sensor_tank_v1-rescue-Uni_General_v1-rescue-Uni_Printer_v1-rescue") (at 78.74 36.83 0) (unit 1)
@@
       (effects (font (size 1.27 1.27)) hide)
     )
+    (pin "1")
+    (pin "2")
+    (pin "3")
+    (pin "4")
+    (pin "5")
+    (pin "6")
+    (pin "7")
+    (pin "8")
   )
   (symbol (lib_id "mfc_base_lib:TLE9251VSJ") (at 77.47 87.63 0) (unit 1)
@@
       (effects (font (size 1.27 1.27)) hide)
     )
+    (pin "1")
+    (pin "2")
+    (pin "3")
+    (pin "4")
+    (pin "5")
+    (pin "6")
+    (pin "7")
+    (pin "8")
   )
 )
