File: Stepdir.kicad_sch (KiCad schematic)
At the start: 2 parts, among them IC2 AM26C31CD

Commit message: Fixes
Signed-off-by: Jarosław Karwik <jaroslaw.karwik@gmail.com>
Parts:
- C26: TME C0603C104K3RAC -> (none)
- IC2: TME (none) -> AM26C31CD
Changed lines of the file:
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@@
       (effects (font (size 1.27 1.27)) hide)
     )
-    (property "TME" "C0603C104K3RAC" (id 4) (at 127 57.15 0)
+    (property "TME" "" (id 4) (at 127 57.15 0)
       (effects (font (size 1.27 1.27)) hide)
     )
@@
       (effects (font (size 1.27 1.27)) (justify left) hide)
     )
+    (property "TME" "AM26C31CD" (id 4) (at 88.9 62.23 0)
+      (effects (font (size 1.27 1.27)) hide)
+    )
   )

Commit message: UPDATE - 3D and Jumper descriptions
Signed-off-by: Jacek <matuszewski.kartech@gmail.com>
Parts:
- C26: TME (none) -> C0603C104K3RAC
Changed lines of the file:
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@@
-(kicad_sch (version 20201015) (generator eeschema)
+(kicad_sch (version 20210126) (generator eeschema)
   (paper "A4")
   (title_block
@@
       (effects (font (size 1.27 1.27)) hide)
     )
+    (pin "1")
   )
   (symbol (lib_id "Uni_Printer-rescue:GND-Sensor_tank_v1-rescue-Uni_General_v1-rescue-Uni_Printer_v1-rescue") (at 71.12 72.39 0) (unit 1)
@@
       (effects (font (size 1.27 1.27)) hide)
     )
+    (pin "1")
   )
   (symbol (lib_id "Uni_Printer-rescue:GND-Sensor_tank_v1-rescue-Uni_General_v1-rescue-Uni_Printer_v1-rescue") (at 86.36 82.55 0) (unit 1)
@@
       (effects (font (size 1.27 1.27)) hide)
     )
+    (pin "1")
   )
   (symbol (lib_id "Uni_Printer-rescue:GND-Sensor_tank_v1-rescue-Uni_General_v1-rescue-Uni_Printer_v1-rescue") (at 114.3 72.39 90) (unit 1)
@@
       (effects (font (size 1.27 1.27)) hide)
     )
+    (pin "1")
   )
   (symbol (lib_id "Uni_Printer-rescue:GND-Sensor_tank_v1-rescue-Uni_General_v1-rescue-Uni_Printer_v1-rescue") (at 130.81 57.15 90) (unit 1)
@@
       (effects (font (size 1.27 1.27)) hide)
     )
+    (pin "1")
   )
   (symbol (lib_id "Uni_Printer-rescue:C-Device") (at 127 57.15 270) (unit 1)
@@
       (effects (font (size 1.27 1.27)) hide)
     )
-    (property "TME" "" (id 4) (at 127 57.15 0)
-      (effects (font (size 1.27 1.27)) hide)
-    )
+    (property "TME" "C0603C104K3RAC" (id 4) (at 127 57.15 0)
+      (effects (font (size 1.27 1.27)) hide)
+    )
+    (pin "1")
+    (pin "2")
   )
   (symbol (lib_id "Uni_Printer-rescue:AM26C31CD-AM26C31CD-Uni_Printer_v1-rescue") (at 88.9 62.23 0) (unit 1)
@@
       (effects (font (size 1.27 1.27)) hide)
     )
+    (pin "1")
+    (pin "10")
+    (pin "11")
+    (pin "12")
+    (pin "13")
+    (pin "14")
+    (pin "15")
+    (pin "16")
+    (pin "2")
+    (pin "3")
+    (pin "4")
+    (pin "5")
+    (pin "6")
+    (pin "7")
+    (pin "8")
+    (pin "9")
   )
 )
