File: Uni_Printer.kicad_pcb (KiCad board)
At the start: 4 copper layers, 81 x 127.6 mm, 179 parts, among them IC1 MAX17503ATP+, IC10 ITS4141NHUMA1, IC11 ITS4141NHUMA1, IC2 AM26C31CD, IC3 74HC14D, IC4 TLV1117-33, IC5 LAN8742A, IC6 ITS4141NHUMA1, IC7 ITS4141NHUMA1, IC8 ITS4141NHUMA1, IC9 ITS4141NHUMA1, J1 Conn_01x10, J10 USB B connector, J11 LMJ1998824110DL1T39J, J12 RJ45, J13 Conn_01x04_Male, J14 Conn_02x13_Odd_Even, J2 Conn_01x10, J3 Conn_01x10, J4 Conn_01x10, J5 FIDUCIAL, J6 FIDUCIAL, J7 Conn_01x10, J8 Conn_01x10, J9 RJ45, SW2 SW_Push, SW3 SW_Push, U1 STM32H743VITx, U3 TLE9251VSJ, U5 ST1480ACDR, U6 ST1480ACDR, U7 ST1480ACDR, U8 ST1480ACDR, U9 ST1480ACDR, Y1 ABM7-8.000MHZ-D2Y-T, Y2 ABM7-25.000MHZ-D2Y-T

Commit message: UPDATE
Signed-off-by: Jacek <matuszewski.kartech@gmail.com>
Parts:
- L1: value 10uH -> 10nH
Connections:
- JP4 pad 2: Net-(JP4-Pad2) -> /IN4
- JP7 pad 2: Net-(JP7-Pad2) -> /SUPPY+
- R21 pad 1: Net-(JP4-Pad2) -> /IN4
- R8 pad 1: Net-(JP7-Pad2) -> /SUPPY+
Routing:
- net /RS485_TX: track 42.2 -> 38.2 mm
- net /ADC.CH1: track 62.1 -> 66.0 mm
- net /ADC.CH2: track 61.1 -> 64.4 mm
- net /IN4: track 8.09 -> 11.3 mm, vias 1 -> 2
- net Net-(JP4-Pad2): track 3.18 -> 0.00 mm, vias 1 -> 0
- net Net-(JP7-Pad2): track 3.01 -> 0.00 mm, vias 1 -> 0
- net /SUPPY+: track 153.0 -> 156.0 mm, vias 1 -> 2

Commit message: Fixes
Signed-off-by: Jarosław Karwik <jaroslaw.karwik@gmail.com>
Parts:
- C1: value 100nF -> 100n
- C10, C11, C13, C23, C38, C8: footprint Capacitor_SMD:C_1206_3216Metric -> Capacitor_SMD:C_0603_1608Metric
- C43: footprint Capacitor_SMD:C_1206_3216Metric -> Capacitor_SMD:C_1210_3225Metric
- C6, C7: value 18p -> 18pF
- CP1: value 1.0uF/1.0ESR -> 2.2uF
- JP1, JP10, JP11, JP12, JP13, JP14, JP15, JP16, JP17, JP18, JP2, JP3, JP4, JP7, JP8, JP9: footprint Jumper:SolderJumper-3_P1.3mm_Bridged2Bar12_RoundedPad1.0x1.5mm -> moje:SolderJumper-3-open
- RN12, RN13: value 15k -> 10k
- U1: value STM32H743VITx -> STM32H743VIT6
- Y1: value ABM7-8.000MHZ-D2Y-T -> ABM7-25.000MHZ-D2Y-T
- moved CP1 6.16 mm to (126.0, 111.5)
- moved C26 4.79 mm to (114.1, 132.2), turned to 180 degrees
- moved C8 4.55 mm to (86.0, 120.0), turned to 0 degrees
- moved C38 3.35 mm to (84.5, 121.8), turned to 0 degrees
- moved C25 3.13 mm to (84.5, 123.4), turned to 0 degrees
- moved RN2 3.03 mm to (122.0, 111.1)
- moved C20 2.66 mm to (128.1, 71.5)
- moved CP2 2.62 mm to (124.4, 111.5), turned to 90 degrees
- moved C10 2.14 mm to (128.0, 73.2)
- moved C34 2.05 mm to (86.0, 118.3), turned to 0 degrees
- moved R49 1.50 mm to (87.2, 56.1)
- moved J6 1.50 mm to (78.0, 141.8)
- moved C24 1.31 mm to (123.3, 91.4)
- moved C27 1.30 mm to (128.4, 127.4), turned to 90 degrees
- moved C11 1.25 mm to (128.0, 74.7)
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Connections:
- net /AIN_IN5 renamed /Digital Inputs/AIN_IN5
- net /AIN_IN6 renamed /Digital Inputs/AIN_IN6
- net /AIN_IN7 renamed /Digital Inputs/AIN_IN7
- net /AIN_IN8 renamed /Digital Inputs/AIN_IN8
- net /AIN_IN_SUP5 renamed /Digital Inputs/AIN_IN_SUP5
- net /AIN_IN_SUP6 renamed /Digital Inputs/AIN_IN_SUP6
- net /AIN_IN_SUP7 renamed /Digital Inputs/AIN_IN_SUP7
- net /AIN_IN_SUP8 renamed /Digital Inputs/AIN_IN_SUP8
- net /DIR1.A renamed /Connectors/DIR1.A
- net /DIR1.B renamed /Connectors/DIR1.B
- net /DIR2.A renamed /Connectors/DIR2.A
- net /DIR2.B renamed /Connectors/DIR2.B
- net /ENC1_IN.A1 renamed /Encoder/ENC1_IN.A1
- net /ENC1_IN.A2 renamed /Encoder/ENC1_IN.A2
- net /ENC1_IN.B1 renamed /Encoder/ENC1_IN.B1
- net /ENC1_IN.B2 renamed /Encoder/ENC1_IN.B2
- net /ENC2_IN.A1 renamed /Encoder/ENC2_IN.A1
- net /ENC2_IN.A2 renamed /Encoder/ENC2_IN.A2
- net /ENC2_IN.B1 renamed /Encoder/ENC2_IN.B1
- net /ENC2_IN.B2 renamed /Encoder/ENC2_IN.B2
- net /ENET_CRSDV renamed /Ethernet/ENET_CRSDV
- net /ENET_MDIO renamed /Ethernet/ENET_MDIO
- net /ENET_REF_CLK renamed /Ethernet/ENET_REF_CLK
- net /ENET_RXD0 renamed /Ethernet/ENET_RXD0
- net /ENET_RXD1 renamed /Ethernet/ENET_RXD1
- net /ETH_MDC__PC1 renamed /Ethernet/ENET_MDC
- net /ETH_TXD0__PB12 renamed /Ethernet/ENET_TXD0
- net /ETH_TXD1__PB13 renamed /Ethernet/ENET_TXD1
- net /ETH_TX_EN__PB11 renamed /Ethernet/ENET_TX_EN
- net /FDCAN_H renamed /Connectors/FDCAN_H
- net /FDCAN_L renamed /Connectors/FDCAN_L
- net /IN1 renamed /Digital Inputs/IN1
- net /IN2 renamed /Digital Inputs/IN2
- net /IN3 renamed /Digital Inputs/IN3
- net /IN_SUP1 renamed /Digital Inputs/IN_SUP1
- net /IN_SUP2 renamed /Digital Inputs/IN_SUP2
- net /IN_SUP3 renamed /Digital Inputs/IN_SUP3
- net /IN_SUP4 renamed /Digital Inputs/IN_SUP4
- net /LPTM1_IN1_PD12 renamed /Processor/LPTM1_IN1_PD12
- net /OUT1 renamed /Outputs/OUT1
- net /OUT2 renamed /Outputs/OUT2
- net /OUT3 renamed /Outputs/OUT3
- net /OUT4 renamed /Outputs/OUT4
- net /OUT5 renamed /Outputs/OUT5
- net /OUT6 renamed /Outputs/OUT6
- net /OUT_E1 renamed /midboard/OUT_E1
- net /OUT_E2 renamed /midboard/OUT_E2
- net /OUT_E3 renamed /midboard/OUT_E3
- net /OUT_E4 renamed /midboard/OUT_E4
- net /OUT_E5 renamed /midboard/OUT_E5
- net /OUT_E6 renamed /midboard/OUT_E6
- net /PWR_RESET renamed /Power_supply/PWR_RESET
- net /RS_485_A renamed /Connectors/RS_485_A
- net /RS_485_B renamed /Connectors/RS_485_B
- net /STEP1.A renamed /Connectors/STEP1.A
- net /STEP1.B renamed /Connectors/STEP1.B
- net /STEP2.A renamed /Connectors/STEP2.A
- net /STEP2.B renamed /Connectors/STEP2.B
- net /TIM16_CH1__PB8 renamed /Processor/TIM16_CH1__PB8
- C40 pad 1: /SUPPY+ -> /Connectors/SUPPY+
- D10 pad 2: /SUPPY+ -> /Connectors/SUPPY+
- D6 pad 1: Net-(D6-Pad1) -> /Processor/D-
- D6 pad 3: Net-(D6-Pad3) -> /Processor/D+
- D6 pad 4: /USB.D+ -> /USB.D-
- D6 pad 6: /USB.D- -> /USB.D+
- IC1 pad 1: /SUPPY+ -> /Connectors/SUPPY+
- IC1 pad 2: /SUPPY+ -> /Connectors/SUPPY+
- IC1 pad 3: /SUPPY+ -> /Connectors/SUPPY+
- IC1 pad 4: /SUPPY+ -> /Connectors/SUPPY+
- IC10 pad 4: /SUPPY+ -> /Connectors/SUPPY+
- IC11 pad 4: /SUPPY+ -> /Connectors/SUPPY+
- IC6 pad 4: /SUPPY+ -> /Connectors/SUPPY+
- IC7 pad 4: /SUPPY+ -> /Connectors/SUPPY+
- IC8 pad 4: /SUPPY+ -> /Connectors/SUPPY+
- IC9 pad 4: /SUPPY+ -> /Connectors/SUPPY+
- J2 pad 10: /SUPPY+ -> /Connectors/SUPPY+
- J2 pad 9: /SUPPY+ -> /Connectors/SUPPY+
- J4 pad 1: /IN4 -> /Digital Inputs/IN4
- JP10 pad 1: /SUPPY+ -> /Connectors/SUPPY+
- JP11 pad 1: /SUPPY+ -> /Connectors/SUPPY+
- JP13 pad 1: /SUPPY+ -> /Connectors/SUPPY+
- JP15 pad 1: /SUPPY+ -> /Connectors/SUPPY+
- JP17 pad 1: /SUPPY+ -> /Connectors/SUPPY+
- JP4 pad 1: /IN4 -> /Digital Inputs/IN4
- JP4 pad 2: /IN4 -> Net-(JP4-Pad2)
- JP7 pad 1: /SUPPY+ -> /Connectors/SUPPY+
- JP7 pad 2: /SUPPY+ -> Net-(JP7-Pad2)
- JP8 pad 1: /SUPPY+ -> /Connectors/SUPPY+
- JP9 pad 1: /SUPPY+ -> /Connectors/SUPPY+
- R18 pad 1: /IN4 -> /Digital Inputs/IN4
- R21 pad 1: /IN4 -> Net-(JP4-Pad2)
- R8 pad 1: /SUPPY+ -> Net-(JP7-Pad2)
- U1 pad 70: Net-(D6-Pad1) -> /Processor/D+
- U1 pad 71: Net-(D6-Pad3) -> /Processor/D-
Routing:
- net +5V: track 352.4 -> 97.6 mm, vias 7 -> 12
- net /SUPPY+: track 156.0 -> 0.00 mm, vias 2 -> 0
- net /Connectors/SUPPY+: track 0.00 -> 77.2 mm, vias 0 -> 12
- net /Processor/D-: track 0.00 -> 40.7 mm
- net Net-(D6-Pad1): track 37.4 -> 0.00 mm
- net Net-(D6-Pad3): track 37.3 -> 0.00 mm
- net /Processor/D+: track 0.00 -> 37.1 mm
- net GND: track 148.1 -> 117.4 mm, vias 124 -> 127
- net +3V3: track 84.0 -> 67.2 mm, vias 46 -> 49
- net /IN4: track 11.3 -> 0.00 mm, vias 2 -> 0
- net /Ethernet/VDD: track 21.8 -> 12.9 mm, vias 19 -> 17
- net /Digital Inputs/IN4: track 0.00 -> 8.09 mm, vias 0 -> 1
- net /Ethernet/VDDCR: track 11.0 -> 4.35 mm
- net /Ethernet/ENET_TXD1: track 87.4 -> 82.2 mm
- net /Ethernet/ENET_TXD0: track 85.3 -> 80.5 mm
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- added copper zone on B.Cu, net +5V
- added copper zone on F.Cu, net +5V
- added copper zone on F.Cu, net /Connectors/SUPPY+
- added copper zone on In2.Cu, net /Connectors/SUPPY+
- removed copper zone on F.Cu, net /SUPPY+
Other:
- board size 81 x 127.6 mm -> 81 x 127.5 mm
- board text added: "+A1-"
- board text added: "+A2-"
- board text added: "+B1-"
- board text added: "+B2-"
- board text added: "+D1-"
- board text added: "+D2-"
- board text added: "+S1-"
- board text added: "+S2-"
- board text added: "LAN"
- board text removed: "A1+"
- board text removed: "A1-"
- board text removed: "A2+"
- board text removed: "A2-"
- board text removed: "B1+"
- board text removed: "B1-"
- board text removed: "B2+"
- board text removed: "B2-"
- board text removed: "D1+"
- board text removed: "D1-"
- board text removed: "D2+"
- board text removed: "D2-"
- board text removed: "S1+"
- board text removed: "S1-"
- board text removed: "S2+"
- board text removed: "S2-"

Commit message: UPDATE - 3D and Jumper descriptions
Signed-off-by: Jacek <matuszewski.kartech@gmail.com>
Parts:
- removed CP1: 2.2uF, Capacitor_SMD:C_0603_1608Metric
- added C39: 2.2uF, Capacitor_SMD:C_0603_1608Metric, F.Cu at (126.0, 111.5)
- JP1: value Jumper -> IN1_P
- JP10: value Jumper -> IN4
- JP11: value Jumper -> IN5
- JP12: value Jumper -> IN5_P
- JP13: value Jumper -> IN6
- JP14: value Jumper -> IN6_P
- JP15: value Jumper -> IN7
- JP16: value Jumper -> IN7_P
- JP17: value Jumper -> IN8
- JP18: value Jumper -> IN8_P
- JP2: value Jumper -> IN2_P
- JP3: value Jumper -> IN3_P
- JP4: value Jumper -> IN4_P
- JP7: value Jumper -> IN1
- JP8: value Jumper -> IN2
- JP9: value Jumper -> IN3
- moved IC2 0.09 mm to (116.2, 126.2)
Connections:
- net /Digital Inputs/AIN_IN5 renamed /Connectors/AIN_IN5
- net /Digital Inputs/AIN_IN6 renamed /Connectors/AIN_IN6
- net /Digital Inputs/AIN_IN7 renamed /Connectors/AIN_IN7
- net /Digital Inputs/AIN_IN8 renamed /Connectors/AIN_IN8
- net /Digital Inputs/AIN_IN_SUP5 renamed /Connectors/AIN_IN_SUP5
- net /Digital Inputs/AIN_IN_SUP6 renamed /Connectors/AIN_IN_SUP6
- net /Digital Inputs/AIN_IN_SUP7 renamed /Connectors/AIN_IN_SUP7
- net /Digital Inputs/AIN_IN_SUP8 renamed /Connectors/AIN_IN_SUP8
- net /Digital Inputs/IN1 renamed /Connectors/IN1
- net /Digital Inputs/IN2 renamed /Connectors/IN2
- net /Digital Inputs/IN3 renamed /Connectors/IN3
- net /Digital Inputs/IN4 renamed /Connectors/IN4
- net /Digital Inputs/IN_SUP1 renamed /Connectors/IN_SUP1
- net /Digital Inputs/IN_SUP2 renamed /Connectors/IN_SUP2
- net /Digital Inputs/IN_SUP3 renamed /Connectors/IN_SUP3
- net /Digital Inputs/IN_SUP4 renamed /Connectors/IN_SUP4
- net /Encoder/ENC1_IN.A1 renamed /Connectors/ENC1_IN.A1
- net /Encoder/ENC1_IN.A2 renamed /Connectors/ENC1_IN.A2
- net /Encoder/ENC1_IN.B1 renamed /Connectors/ENC1_IN.B1
- net /Encoder/ENC1_IN.B2 renamed /Connectors/ENC1_IN.B2
- net /Encoder/ENC2_IN.A1 renamed /Connectors/ENC2_IN.A1
- net /Encoder/ENC2_IN.A2 renamed /Connectors/ENC2_IN.A2
- net /Encoder/ENC2_IN.B1 renamed /Connectors/ENC2_IN.B1
- net /Encoder/ENC2_IN.B2 renamed /Connectors/ENC2_IN.B2
- net /Outputs/OUT1 renamed /Connectors/OUT_HSW1
- net /Outputs/OUT2 renamed /Connectors/OUT_HSW2
- net /Outputs/OUT3 renamed /Connectors/OUT_HSW3
- net /Outputs/OUT4 renamed /Connectors/OUT_HSW4
- net /Outputs/OUT5 renamed /Connectors/OUT_HSW5
- net /Outputs/OUT6 renamed /Connectors/OUT_HSW6
- net /midboard/OUT_E1 renamed /Analod / Digital IO/OUT_E1
- net /midboard/OUT_E2 renamed /Analod / Digital IO/OUT_E2
- net /midboard/OUT_E3 renamed /Analod / Digital IO/OUT_E3
- net /midboard/OUT_E4 renamed /Analod / Digital IO/OUT_E4
- net /midboard/OUT_E5 renamed /Analod / Digital IO/OUT_E5
- net /midboard/OUT_E6 renamed /Analod / Digital IO/OUT_E6
Routing:
- net GND: track 117.4 -> 119.3 mm
- net +5V: track 97.6 -> 98.9 mm
Other:
- board text added: "IN1"
- board text added: "IN1_P"
- board text added: "IN2"
- board text added: "IN2_P"
- board text added: "IN3"
- board text added: "IN3_P"
- board text added: "IN4"
- board text added: "IN4_P"
- board text added: "IN5"
- board text added: "IN5_P"
- board text added: "IN6"
- board text added: "IN6_P"
- board text added: "IN7"
- board text added: "IN7_P"
- board text added: "IN8"
- board text added: "IN8_P"
