File: ethernet.kicad_sch (KiCad schematic)
At the start: 25 parts, among them IC5 LAN8742A, J11 LMJ1998824110DL1T39J, Y2 ABM7-25.000MHZ-D2Y-T

Commit message: UPDATE - Traces finished
Signed-off-by: Jacek <matuszewski.kartech@gmail.com>
Parts:
- L1: value 10uH -> 10nH
Changed lines of the file:
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@@
     (in_bom yes) (on_board yes)
     (property "Reference" "L1" (id 0) (at 167.64 46.99 0))
-    (property "Value" "10uH" (id 1) (at 167.64 50.8 0))
+    (property "Value" "10nH" (id 1) (at 167.64 50.8 0))
     (property "Footprint" "Inductor_SMD:L_0603_1608Metric" (id 2) (at 167.64 49.53 0)
       (effects (font (size 1.27 1.27)) hide)

Commit message: Fixes
Signed-off-by: Jarosław Karwik <jaroslaw.karwik@gmail.com>
Parts:
- C4, C5: TME VJ0603A180JXACW2BC -> (none)
- C6, C7: value 18p -> 18pF
- CP1: value 1.0uF/1.0ESR -> 2.2uF
- CP2: TME (none) -> 0603B471K101CT
- IC5: TME (none) -> LAN8742A-CZ
- L1: TME (none) -> LQW18AN10NJ00D
- RN10, RN3: TME (none) -> DR1206-390K-4/8
- RN2: TME (none) -> DR1206-10K-4/8
- Y2: Category (none) -> Xtal
Changed lines of the file:
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@@
     )
     (property "Datasheet" "" (id 3) (at 167.64 49.53 0))
+    (property "TME" "LQW18AN10NJ00D" (id 4) (at 167.64 49.53 0)
+      (effects (font (size 1.27 1.27)) hide)
+    )
   )
   (symbol (lib_id "step2cnc-rescue:R-RESCUE-step2cnc8_") (at 66.04 101.6 90) (mirror x) (unit 1)
@@
       (effects (font (size 1.27 1.27)) hide)
     )
-    (property "TME" "VJ0603A180JXACW2BC" (id 4) (at 76.2 110.49 90)
+    (property "TME" "" (id 4) (at 76.2 110.49 90)
       (effects (font (size 1.27 1.27)) hide)
     )
@@
       (effects (font (size 1.27 1.27)) hide)
     )
-    (property "TME" "VJ0603A180JXACW2BC" (id 4) (at 76.2 121.92 90)
+    (property "TME" "" (id 4) (at 76.2 121.92 90)
       (effects (font (size 1.27 1.27)) hide)
     )
@@
       (effects (font (size 1.27 1.27)) (justify left))
     )
-    (property "Value" "18p" (id 1) (at 141.605 137.16 0)
+    (property "Value" "18pF" (id 1) (at 141.605 137.16 0)
       (effects (font (size 1.27 1.27)) (justify left))
     )
@@
       (effects (font (size 1.27 1.27)) (justify left))
     )
-    (property "Value" "18p" (id 1) (at 150.495 137.16 0)
+    (property "Value" "18pF" (id 1) (at 150.495 137.16 0)
       (effects (font (size 1.27 1.27)) (justify left))
     )
@@
       (effects (font (size 1.27 1.27)) (justify left))
     )
-    (property "Value" "1.0uF/1.0ESR" (id 1) (at 168.275 137.16 0)
+    (property "Value" "2.2uF" (id 1) (at 168.275 137.16 0)
       (effects (font (size 1.27 1.27)) (justify left))
     )
@@
       (effects (font (size 1.27 1.27)) hide)
     )
+    (property "TME" "0603B471K101CT" (id 4) (at 176.53 134.62 0)
+      (effects (font (size 1.27 1.27)) hide)
+    )
   )
   (symbol (lib_id "Device:C") (at 185.42 134.62 180) (unit 1)
@@
     )
     (property "TME" "ABM7-25.000MHZ-D2Y" (id 4) (at 82.55 116.84 90)
+      (effects (font (size 1.27 1.27)) hide)
+    )
+    (property "Category" "Xtal" (id 4) (at 82.55 116.84 0)
       (effects (font (size 1.27 1.27)) hide)
     )
@@
       (effects (font (size 1.27 1.27)) hide)
     )
+    (property "TME" "DR1206-10K-4/8" (id 4) (at 72.39 59.69 0)
+      (effects (font (size 1.27 1.27)) hide)
+    )
   )
   (symbol (lib_id "Device:R_Pack04") (at 88.9 59.69 180) (unit 1)
@@
       (effects (font (size 1.27 1.27)) hide)
     )
+    (property "TME" "DR1206-390K-4/8" (id 4) (at 88.9 59.69 0)
+      (effects (font (size 1.27 1.27)) hide)
+    )
   )
   (symbol (lib_id "Device:R_Pack04") (at 161.29 101.6 270) (unit 1)
@@
       (effects (font (size 1.27 1.27)) hide)
     )
+    (property "TME" "DR1206-390K-4/8" (id 4) (at 161.29 101.6 0)
+      (effects (font (size 1.27 1.27)) hide)
+    )
   )
   (symbol (lib_id "Uni_Printer-rescue:RJ45-TRANSFO_v2-rj12") (at 278.13 78.74 0) (unit 1)
@@
       (effects (font (size 1.27 1.27)) hide)
     )
+    (property "TME" "LAN8742A-CZ" (id 4) (at 133.35 88.9 0)
+      (effects (font (size 1.27 1.27)) hide)
+    )

Commit message: UPDATE - 3D and Jumper descriptions
Signed-off-by: Jacek <matuszewski.kartech@gmail.com>
Parts:
- removed CP1: 2.2uF, Capacitor_SMD:C_0603_1608Metric, symbol Device:CP1
- added C39: 2.2uF, Capacitor_SMD:C_0603_1608Metric, symbol Device:C_Small
- C21, C33, C35, C36, C37: TME (none) -> C0603C104K3RAC
- C4, C5, C6, C7: TME (none) -> 0603N180G500CT
- C9: TME (none) -> CL10A106MQ8NNNC
- R1: TME (none) -> WF06P-33R-5%
- R38: TME (none) -> SMD0603-12.1K-1%
- R45, R46, R47, R48: TME (none) -> SMD0603-49R9-1%
Connections:
- net GND: now also C39.2
- net VDDCR: now also C39.1
