File: processor.kicad_sch (KiCad schematic)
At the start: 29 parts, among them J13 Conn_01x04_Male, SW2 SW_Push, SW3 SW_Push, U1 STM32H743VITx, Y1 ABM7-8.000MHZ-D2Y-T

Commit message: Fixes
Signed-off-by: Jarosław Karwik <jaroslaw.karwik@gmail.com>
Parts:
- C10, C11, C13, C23: footprint Capacitor_SMD:C_1206_3216Metric -> Capacitor_SMD:C_0603_1608Metric; TME 0805X106K100CT -> (none)
- C12, C14, C15, C17, C20, C22, C24: TME C0603C104K3RAC -> (none)
- C18, C19: TME VJ0603A180JXACW2BC -> (none)
- D6: TME (none) -> NUF2042XV6T1G
- R4, R5: TME HP03-2K25% -> (none)
- RN1, RN8: TME (none) -> DR1206-100R-4/8
- RN5: TME DR1206-390K-4/8 -> DR1206-100R-4/8
- U1: value STM32H743VITx -> STM32H743VIT6; Category (none) -> Processor; Digi (none) -> 497-17720-ND
- Y1: value ABM7-8.000MHZ-D2Y-T -> ABM7-25.000MHZ-D2Y-T; Category (none) -> Xtal; TME ABM7-8.000MHZ-D2Y -> ABM7-25.000MHZ-D2Y
Connections:
- net USB_DM__PA11: now also D6.4 (D2_2); no longer D6.6 (D1_2)
- net USB_DP__PA12: now also D6.6 (D1_2); no longer D6.4 (D2_2)
- net D+: now reaches U1.70 (PA11)
- net D+: now also D6.3 (D2_1); no longer D6.1 (D1_1)
- net D-: now reaches U1.71 (PA12)
- net D-: now also D6.1 (D1_1); no longer D6.3 (D2_1)

Commit message: UPDATE - 3D and Jumper descriptions
Signed-off-by: Jacek <matuszewski.kartech@gmail.com>
Parts:
- C10, C11, C13, C23: TME (none) -> CL10A106MQ8NNNC
- C12, C14, C15, C16, C17, C20, C22, C24: TME (none) -> C0603C104K3RAC
- C18, C19: TME (none) -> 0603N180G500CT
- D2, D3, D9: TME (none) -> LL-S170PGC-G5-1A
- R3, R4, R5: TME (none) -> HP03-2K25%
