File: hardware/00_main_unit/Analog_digital_io.kicad_sch (KiCad schematic)
At the start: 4 parts, among them IC3 74HC14D

Commit message: Fixes after wrong merge
Signed-off-by: Jacek <matuszewski.kartech@gmail.com>
Parts:
- C31: TME C0603C104K3RAC -> (none)
Changed lines of the file:
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@@
-      (effects (font (size 1.27 1.27)) hide)
-    )
-    (property "TME" "C0603C104K3RAC" (id 4) (at 128.905 52.07 0)
       (effects (font (size 1.27 1.27)) hide)
     )
