File: hardware/00_main_unit/Encoder.kicad_sch (KiCad schematic)
At the start: 12 parts, among them U5 ST1480ACDR, U6 ST1480ACDR, U7 ST1480ACDR, U8 ST1480ACDR

Commit message: Fixes after wrong merge
Signed-off-by: Jacek <matuszewski.kartech@gmail.com>
Parts:
- C27, C28, C29, C30: TME C0603C104K3RAC -> (none)
- R22, R23, R24, R25: TME WF06P-120R-5% -> (none)
Changed lines of the file:
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@@
       (effects (font (size 1.27 1.27)) hide)
     )
-    (property "TME" "WF06P-120R-5%" (id 4) (at 120.65 120.65 0)
+    (property "TME" "" (id 4) (at 120.65 120.65 0)
       (effects (font (size 1.27 1.27)) hide)
     )
@@
       (effects (font (size 1.27 1.27)) hide)
     )
-    (property "TME" "WF06P-120R-5%" (id 4) (at 121.92 76.2 0)
+    (property "TME" "" (id 4) (at 121.92 76.2 0)
       (effects (font (size 1.27 1.27)) hide)
     )
@@
       (effects (font (size 1.27 1.27)) hide)
     )
-    (property "TME" "WF06P-120R-5%" (id 4) (at 199.39 119.38 0)
+    (property "TME" "" (id 4) (at 199.39 119.38 0)
       (effects (font (size 1.27 1.27)) hide)
     )
@@
       (effects (font (size 1.27 1.27)) hide)
     )
-    (property "TME" "WF06P-120R-5%" (id 4) (at 200.66 74.93 0)
+    (property "TME" "" (id 4) (at 200.66 74.93 0)
       (effects (font (size 1.27 1.27)) hide)
     )
@@
       (effects (font (size 1.27 1.27)) hide)
     )
-    (property "TME" "C0603C104K3RAC" (id 4) (at 114.3 58.42 0)
+    (property "TME" "" (id 4) (at 114.3 58.42 0)
       (effects (font (size 1.27 1.27)) hide)
     )
@@
       (effects (font (size 1.27 1.27)) hide)
     )
-    (property "TME" "C0603C104K3RAC" (id 4) (at 114.3 102.87 0)
+    (property "TME" "" (id 4) (at 114.3 102.87 0)
       (effects (font (size 1.27 1.27)) hide)
     )
@@
       (effects (font (size 1.27 1.27)) hide)
     )
-    (property "TME" "C0603C104K3RAC" (id 4) (at 193.04 57.15 0)
-      (effects (font (size 1.27 1.27)) hide)
-    )
     (pin "1")
     (pin "2")
@@
       (effects (font (size 1.27 1.27)) hide)
     )
-    (property "TME" "C0603C104K3RAC" (id 4) (at 193.04 101.6 0)
+    (property "TME" "" (id 4) (at 193.04 101.6 0)
       (effects (font (size 1.27 1.27)) hide)
     )
