File: hardware/00_main_unit/Encoder.kicad_sch (KiCad schematic)
At the start: 12 parts, among them U5 ST1480ACDR, U6 ST1480ACDR, U7 ST1480ACDR, U8 ST1480ACDR

Commit message: FW and SW updates for new revision
Signed-off-by: Jarosław Karwik <jaroslaw.karwik@gmail.com>
Parts:
- removed C29, C30: 100n, Capacitor_SMD:C_0603_1608Metric, symbol Uni_Printer-rescue:C_Small-Device
- removed U5, U6, U7, U8: ST1480ACDR, moje:SOIC-8_3.9x4.9mm_P1.27mm, symbol Uni_Printer-rescue:ST1480ACDR-Sensor_tank_v1-rescue-Uni_General_v1-rescue-Uni_P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
- added R39, R40, R50, R51: 120R, Resistor_SMD:R_0603_1608Metric, symbol Uni_Printer-rescue:R-Device
- added U3, U4: AM26LV32xNS, Package_SO:SOIC-16W_5.3x10.2mm_P1.27mm, symbol Interface:AM26LV32xNS
Connections:
- net ENC1.CH1: now also U3.3 (1Y)
- net ENC1.CH2: now also U3.5 (2Y)
- net ENC1_IN.A1: now also R25.1, U3.2 (1A); no longer R23.1
- net ENC1_IN.A2: now also R23.2, U3.6 (2A); no longer R22.1
- net ENC1_IN.B1: now also R25.2, U3.1 (1B); no longer R23.2
- net ENC1_IN.B2: now also R23.1, U3.7 (2B); no longer R22.2
- net ENC2.CH1: now also U3.11 (3Y)
- net ENC2.CH2: now also U3.13 (4Y)
- net ENC2_IN.A1: now also R22.2, U3.10 (3A); no longer R25.1
- net ENC2_IN.A2: now also R24.2, U3.14 (4A); no longer R24.1
- net ENC2_IN.B1: now also R22.1, U3.9 (3B); no longer R25.2
- net ENC2_IN.B2: now also R24.1, U3.15 (4B); no longer R24.2
- net GND: now also U3.12 (~{G}), U3.4 (G), U3.8 (GND), U4.12 (~{G}), U4.4 (G), U4.8 (GND)
- net +3V3 renamed +5V
- net +5V: now also U3.16 (VDD), U4.16 (VDD)
- new net DIFF_IN.A1: R40.2, U4.10 (3A)
- new net DIFF_IN.A2: R51.2, U4.14 (4A)
- new net DIFF_IN.B1: R40.1, U4.9 (3B)
- new net DIFF_IN.B2: R51.1, U4.15 (4B)
- new net ENC3.CH1: U4.3 (1Y)
- new net ENC3.CH2: U4.5 (2Y)
- new net ENC3_IN.A1: R39.1, U4.2 (1A)
- new net ENC3_IN.A2: R50.2, U4.6 (2A)
- new net ENC3_IN.B1: R39.2, U4.1 (1B)
- new net ENC3_IN.B2: R50.1, U4.7 (2B)
- new net IN_CPU10: U4.13 (4Y)
- new net IN_CPU9: U4.11 (3Y)
- no-connect marks 4 -> 0
Other:
- moved on the sheet: C27, R22, R23, R24, R25
