File: hardware/00_main_unit/midboard.kicad_sch (KiCad schematic)
At the start: 7 parts, among them J14 Conn_02x13_Odd_Even

Commit message: Fixes after wrong merge
Signed-off-by: Jacek <matuszewski.kartech@gmail.com>
Parts:
- C25, C34: TME C0603C104K3RAC -> (none)
- C38, C8: TME CL10A106MQ8NNNC -> (none)
Changed lines of the file:
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@@
       (effects (font (size 1.27 1.27)) hide)
     )
-    (property "TME" "C0603C104K3RAC" (id 4) (at 158.75 82.55 0)
+    (property "TME" "" (id 4) (at 158.75 82.55 0)
       (effects (font (size 1.27 1.27)) hide)
     )
@@
       (effects (font (size 1.27 1.27)) hide)
     )
-    (property "TME" "C0603C104K3RAC" (id 4) (at 219.71 82.55 0)
+    (property "TME" "" (id 4) (at 219.71 82.55 0)
       (effects (font (size 1.27 1.27)) hide)
     )
@@
       (effects (font (size 1.27 1.27)) hide)
     )
-    (property "TME" "CL10A106MQ8NNNC" (id 4) (at 151.13 82.55 0)
+    (property "TME" "" (id 4) (at 151.13 82.55 0)
       (effects (font (size 1.27 1.27)) hide)
     )
@@
       (effects (font (size 1.27 1.27)) hide)
     )
-    (property "TME" "CL10A106MQ8NNNC" (id 4) (at 227.33 82.55 0)
+    (property "TME" "" (id 4) (at 227.33 82.55 0)
       (effects (font (size 1.27 1.27)) hide)
     )
