File: hardware/00_main_unit/RS485_CAN.kicad_sch (KiCad schematic)
At the start: 9 parts, among them U3 TLE9251VSJ, U9 ST1480ACDR

Commit message: Fixes after wrong merge
Signed-off-by: Jacek <matuszewski.kartech@gmail.com>
Parts:
- C2, C3, C32: TME C0603C104K3RAC -> (none)
- R39, R40: TME WF06P-120R-5% -> (none)
Changed lines of the file:
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@@
       (effects (font (size 1.27 1.27)) hide)
     )
-    (property "TME" "WF06P-120R-5%" (id 4) (at 105.41 49.53 90)
+    (property "TME" "" (id 4) (at 105.41 49.53 90)
       (effects (font (size 1.27 1.27)) hide)
     )
@@
       (effects (font (size 1.27 1.27)) hide)
     )
-    (property "TME" "WF06P-120R-5%" (id 4) (at 105.41 96.52 90)
+    (property "TME" "" (id 4) (at 105.41 96.52 90)
       (effects (font (size 1.27 1.27)) hide)
     )
@@
       (effects (font (size 1.27 1.27)) hide)
     )
-    (property "TME" "C0603C104K3RAC" (id 4) (at 83.82 26.67 0)
+    (property "TME" "" (id 4) (at 83.82 26.67 0)
       (effects (font (size 1.27 1.27)) hide)
     )
@@
       (effects (font (size 1.524 1.524)) hide)
     )
-    (property "TME" "C0603C104K3RAC" (id 4) (at 36.83 69.85 0)
-      (effects (font (size 1.27 1.27)) hide)
-    )
     (pin "1")
     (pin "2")
@@
       (effects (font (size 1.524 1.524)) hide)
     )
-    (property "TME" "C0603C104K3RAC" (id 4) (at 52.07 69.85 0)
-      (effects (font (size 1.27 1.27)) hide)
-    )
     (pin "1")
