File: hardware/00_main_unit/Uni_Printer.kicad_pcb (KiCad board)
At the start: 4 copper layers, 81 x 127.5 mm, 182 parts, among them IC1 MAX17503ATP+, IC10 ITS4141NHUMA1, IC11 ITS4141NHUMA1, IC2 AM26C31CD, IC3 74HC14D, IC4 TLV1117-33, IC5 LAN8742A, IC6 ITS4141NHUMA1, IC7 ITS4141NHUMA1, IC8 ITS4141NHUMA1, IC9 ITS4141NHUMA1, J1 Conn_01x10, J10 USB B connector, J11 LMJ1998824110DL1T39J, J12 RJ45, J13 Conn_01x04_Male, J14 Conn_02x15_Odd_Even, J15 Conn_01x06_Male, J2 Conn_01x10, J3 Conn_01x10, J4 Conn_01x10, J5 FIDUCIAL, J6 FIDUCIAL, J7 Conn_01x10, J8 Conn_01x10, J9 RJ45, SW2 SW_Push, SW3 SW_Push, U1 STM32H743VIT6, U3 TLE9251VSJ, U5 ST1480ACDR, U6 ST1480ACDR, U7 ST1480ACDR, U8 ST1480ACDR, U9 ST1480ACDR, Y1 ABM7-25.000MHZ-D2Y-T, Y2 ABM7-25.000MHZ-D2Y-T

Commit message: FW and SW updates for new revision
Signed-off-by: Jarosław Karwik <jaroslaw.karwik@gmail.com>
Parts:
- removed C29, C30, C31, C32, C34: 100n, Capacitor_SMD:C_0603_1608Metric
- removed C38: 10uF, Capacitor_SMD:C_0603_1608Metric
- removed D1: D_Schottky_x4_BAV99S, moje:SOT-363
- removed JP5, JP6: Jumper, Jumper:SolderJumper-2_P1.3mm_Open_RoundedPad1.0x1.5mm
- removed RN4, RN9: 100R, moje:R_Array_Convex_4x0603
- removed SW2, SW3: SW_Push, Buttons_Switches_SMD:SW_SPST_B3U-1000P
- removed U5, U6, U7, U8, U9: ST1480ACDR, moje:SOIC-8_3.9x4.9mm_P1.27mm
- added IC12: AM26C31CD, moje:SOIC127P600X175-16N, F.Cu at (106.5, 137.1)
- added IC13: AM26C31CD, moje:SOIC127P600X175-16N, F.Cu at (98.0, 137.1)
- added J16: RJ45_Shielded, Connector_RJ:RJ45_Ninigi_GE, F.Cu at (144.6, 139.7)
- added J17: RJ45_Shielded, Connector_RJ:RJ45_Ninigi_GE, F.Cu at (88.4, 81.5)
- added J18: RJ45_Shielded, Connector_RJ:RJ45_Ninigi_GE, F.Cu at (88.3, 61.4)
- added R50: 120R, Resistor_SMD:R_0603_1608Metric, F.Cu at (122.5, 145.2)
- added R51: 120R, Resistor_SMD:R_0603_1608Metric, F.Cu at (130.5, 142.7)
- added U2: P82B96, Package_SO:TSSOP-8_4.4x3mm_P0.65mm, F.Cu at (133.6, 143.4)
- added U4: AM26LV32xNS, Package_SO:SOIC-16W_5.3x10.2mm_P1.27mm, F.Cu at (125.5, 135.5)
- C8: value 10uF -> 100n
- IC3: value 74HC14D -> AM26C31CD; footprint moje:SO14 -> moje:SOIC127P600X175-16N
- J12: value RJ45 -> Conn_02x07_Odd_Even; footprint Connector_RJ:RJ45_Amphenol_54602-x08_Horizontal -> Connector_PinHeader_2.54mm:PinHeader_2x07_P2.54mm_Vertical
- J14: value Conn_02x15_Odd_Even -> Conn_01x10; footprint Connector_PinHeader_2.54mm:PinHeader_2x15_P2.54mm_Vertical -> moje:PhoenixContact_MC-G_10x3.50mm_Angled
- J9: value RJ45 -> Conn_02x02_Odd_Even; footprint Connector_RJ:RJ45_Amphenol_54602-x08_Horizontal -> Connector_PinHeader_2.54mm:PinHeader_2x02_P2.54mm_Vertical
- U3: value TLE9251VSJ -> AM26LV32xNS; footprint Package_SO:SOIC-8_3.9x4.9mm_P1.27mm -> Package_SO:SOIC-16W_5.3x10.2mm_P1.27mm
- moved C3 86.4 mm to (87.2, 144.1)
- moved R40 86.2 mm to (122.5, 142.7), turned to 0 degrees
- moved U3 81.0 mm to (135.7, 135.5), turned to 0 degrees
- moved C2 76.7 mm to (117.2, 137.2), turned to 0 degrees
- moved R39 71.8 mm to (126.5, 142.7), turned to 0 degrees
- moved IC3 38.0 mm to (89.5, 137.1), turned to 0 degrees
- moved C8 24.6 mm to (91.2, 144.1)
- moved C25 23.4 mm to (87.2, 146.6)
- moved C28 20.5 mm to (126.5, 145.2), turned to 0 degrees
- moved J12 19.8 mm to (95.0, 63.9), turned to 90 degrees
- moved J9 18.6 mm to (99.3, 76.3), turned to 0 degrees
- moved J7 13.3 mm to (121.7, 149.3)
- moved J8 13.3 mm to (81.1, 149.3)
- moved J14 10.8 mm to (79.9, 107.2), turned to -90 degrees
Connections:
- C25 pad 1: +5V -> GND
- C25 pad 2: GND -> +5V
- C27 pad 1: +3V3 -> +5V
- C28 pad 1: +3V3 -> +5V
- C3 pad 1: +3V3 -> GND
- C3 pad 2: GND -> +5V
- C8 pad 1: +3V3 -> GND
- C8 pad 2: GND -> +5V
- IC3 pad 1: /OUT_STEP1 -> /OUT_STEP3
- IC3 pad 10: Net-(IC3-Pad10) -> /Connectors/DIR4.A
- IC3 pad 11: /OUT_STEP3 -> /Connectors/DIR4.B
- IC3 pad 12: Net-(IC3-Pad12) -> GND
- IC3 pad 13: /OUT_DIR3 -> /Connectors/STEP4.B
- IC3 pad 14: +5V -> /Connectors/STEP4.A
- IC3 pad 2: Net-(IC3-Pad2) -> /Connectors/STEP3.A
- IC3 pad 3: /OUT_DIR1 -> /Connectors/STEP3.B
- IC3 pad 4: Net-(IC3-Pad4) -> GND
- IC3 pad 5: /OUT_STEP2 -> /Connectors/DIR3.B
- IC3 pad 6: Net-(IC3-Pad6) -> /Connectors/DIR3.A
- IC3 pad 7: GND -> /OUT_DIR3
- IC3 pad 8: Net-(IC3-Pad8) -> GND
- IC3 pad 9: /OUT_DIR2 -> /OUT_DIR4
- J12 pad 1: /Connectors/FDCAN_H -> /Analog  Digital IO/OUT_EXT_STEP1
- J12 pad 2: /Connectors/FDCAN_L -> /Analog  Digital IO/OUT_EXT_DIR1
- J12 pad 3: GND -> /Analog  Digital IO/OUT_EXT_STEP2
- J12 pad 4: GND -> /Analog  Digital IO/OUT_EXT_DIR2
- J12 pad 5: GND -> /Analog  Digital IO/OUT_EXT_STEP3
- J12 pad 6: GND -> /Analog  Digital IO/OUT_EXT_DIR3
- J12 pad 7: /Connectors/RS_485_A -> /Analog  Digital IO/OUT_EXT_STEP8
- J12 pad 8: /Connectors/RS_485_B -> /Analog  Digital IO/OUT_EXT_DIR8
- J14 pad 1: /midboard/RES_UART.TX -> +5V
- J14 pad 10: /I2C.SDA -> /Connectors/DIR3.B
- J14 pad 2: /midboard/RES_UART.RX -> /Connectors/ENC3_IN.A1
- J14 pad 3: /Analod / Digital IO/OUT_E1 -> /Connectors/ENC3_IN.B1
- J14 pad 4: /Analod / Digital IO/OUT_E2 -> /Connectors/ENC3_IN.A2
- J14 pad 5: /Analod / Digital IO/OUT_E3 -> /Connectors/ENC3_IN.B2
- J14 pad 6: /Analod / Digital IO/OUT_E4 -> GND
- J14 pad 7: /Analod / Digital IO/OUT_E5 -> /Connectors/STEP3.A
- J14 pad 8: /Analod / Digital IO/OUT_E6 -> /Connectors/STEP3.B
- J14 pad 9: /I2C.SCL -> /Connectors/DIR3.A
- J9 pad 1: /Connectors/FDCAN_H -> GND
- J9 pad 2: /Connectors/FDCAN_L -> /Processor/NRST
- J9 pad 3: GND -> +3V3
- J9 pad 4: GND -> /Processor/BOOT0
- R22 pad 1: /Connectors/ENC1_IN.A2 -> /Connectors/ENC2_IN.B1
- R22 pad 2: /Connectors/ENC1_IN.B2 -> /Connectors/ENC2_IN.A1
- R23 pad 1: /Connectors/ENC1_IN.A1 -> /Connectors/ENC1_IN.B2
- R23 pad 2: /Connectors/ENC1_IN.B1 -> /Connectors/ENC1_IN.A2
- R24 pad 1: /Connectors/ENC2_IN.A2 -> /Connectors/ENC2_IN.B2
- R24 pad 2: /Connectors/ENC2_IN.B2 -> /Connectors/ENC2_IN.A2
- R25 pad 1: /Connectors/ENC2_IN.A1 -> /Connectors/ENC1_IN.A1
- R25 pad 2: /Connectors/ENC2_IN.B1 -> /Connectors/ENC1_IN.B1
- R39 pad 1: Net-(JP5-Pad1) -> /Connectors/ENC3_IN.A1
- R39 pad 2: /Connectors/RS_485_B -> /Connectors/ENC3_IN.B1
- R40 pad 1: Net-(JP6-Pad1) -> /Connectors/DIFF_IN.B1
- R40 pad 2: /Connectors/FDCAN_L -> /Connectors/DIFF_IN.A1
- RN6 pad 1: Net-(IC3-Pad6) -> /OUT_STEP2
- RN6 pad 2: Net-(IC3-Pad4) -> /OUT_DIR1
- RN6 pad 3: Net-(IC3-Pad2) -> /OUT_STEP1
- RN6 pad 4: unconnected-(RN6-Pad4) -> /OUT_STEP8
- RN6 pad 5: unconnected-(RN6-Pad5) -> /Analog  Digital IO/OUT_EXT_STEP8
- RN6 pad 6: /Analod / Digital IO/OUT_E1 -> /Analog  Digital IO/OUT_EXT_STEP1
- RN6 pad 7: /Analod / Digital IO/OUT_E2 -> /Analog  Digital IO/OUT_EXT_DIR1
- RN6 pad 8: /Analod / Digital IO/OUT_E3 -> /Analog  Digital IO/OUT_EXT_STEP2
- RN7 pad 1: Net-(IC3-Pad8) -> /OUT_DIR2
- RN7 pad 2: Net-(IC3-Pad10) -> /OUT_STEP3
- RN7 pad 3: Net-(IC3-Pad12) -> /OUT_DIR3
- RN7 pad 4: unconnected-(RN7-Pad4) -> /OUT_DIR8
- RN7 pad 5: unconnected-(RN7-Pad5) -> /Analog  Digital IO/OUT_EXT_DIR8
- RN7 pad 6: /Analod / Digital IO/OUT_E6 -> /Analog  Digital IO/OUT_EXT_DIR3
- RN7 pad 7: /Analod / Digital IO/OUT_E5 -> /Analog  Digital IO/OUT_EXT_STEP3
- RN7 pad 8: /Analod / Digital IO/OUT_E4 -> /Analog  Digital IO/OUT_EXT_DIR2
- U1 pad 1: /SPI.SCLK -> /OUT_STEP5
- U1 pad 25: /RS485_TX -> unconnected-(U1-Pad25)
- U1 pad 3: /SPI.NSS -> /OUT_DIR6
- U1 pad 4: /SPI.MISO -> /OUT_DIR5
- U1 pad 44: /MID_IO.IO1 -> /IN_CPU10
- U1 pad 45: /MID_IO.IO2 -> /IN_CPU9
- U1 pad 5: /SPI.MOSI -> /OUT_STEP6
- U1 pad 59: /MID_IO.IO3_DIR4 -> /OUT_STEP4
- U1 pad 68: /UART.TX -> /OUT_STEP7
- U1 pad 69: /UART.RX -> /OUT_DIR7
- U1 pad 77: /TIM.CH1 -> /ENC3.CH1
- U1 pad 81: /FDCAN_RX -> unconnected-(U1-Pad81)
- U1 pad 82: /FDCAN_TX -> /OUT_STEP8
- U1 pad 83: unconnected-(U1-Pad83) -> /OUT_DIR8
- U1 pad 85: /RS485_DE -> unconnected-(U1-Pad85)
- U1 pad 86: /RS485_RX -> unconnected-(U1-Pad86)
- U1 pad 89: /TIM.CH2 -> /ENC3.CH2
- U1 pad 95: /MID_IO.IO4_STEP4 -> /OUT_DIR4
- U3 pad 1: /FDCAN_TX -> /Connectors/ENC1_IN.B1
- U3 pad 2: GND -> /Connectors/ENC1_IN.A1
- U3 pad 3: +5V -> /ENC1.CH1
- U3 pad 4: /FDCAN_RX -> GND
- U3 pad 5: +3V3 -> /ENC1.CH2
- U3 pad 6: /Connectors/FDCAN_L -> /Connectors/ENC1_IN.A2
- U3 pad 7: /Connectors/FDCAN_H -> /Connectors/ENC1_IN.B2
Routing:
- net GND: track 122.7 -> 319.3 mm, vias 128 -> 129
- net /I2C.SDA: track 69.3 -> 206.6 mm, vias 2 -> 8
- net /OUT_STEP5: track 0.00 -> 116.3 mm, vias 0 -> 2
- net /Connectors/ENC3_IN.A1: track 0.00 -> 95.2 mm, vias 0 -> 2
- net /OUT_STEP7: track 0.00 -> 90.7 mm, vias 0 -> 2
- net /Connectors/STEP3.B: track 0.00 -> 79.6 mm, vias 0 -> 3
- net /TIM.CH1: track 79.1 -> 0.00 mm, vias 2 -> 0
- net /ENC3.CH1: track 0.00 -> 79.1 mm, vias 0 -> 2
- net /MID_IO.IO3_DIR4: track 76.9 -> 0.00 mm, vias 2 -> 0
- net /MID_IO.IO1: track 74.0 -> 0.00 mm, vias 1 -> 0
- net /Connectors/ENC3_IN.A2: track 0.00 -> 74.0 mm, vias 0 -> 1
- net /MID_IO.IO2: track 72.0 -> 0.00 mm, vias 1 -> 0
- net /IN_CPU9: track 0.00 -> 72.0 mm, vias 0 -> 1
- net /I2C.SCL: track 71.1 -> 0.00 mm, vias 3 -> 0
- net /UART.TX: track 71.0 -> 0.00 mm, vias 2 -> 0
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Other:
- board text added: "UNI CTRL 4.0"
- board text removed: "UNI CTRL 3.1"
