File: hardware/10_shield_stick_head/Uni_stick.kicad_pcb (KiCad board)
At the start: 2 copper layers, 68.4 x 95.8 mm, 52 parts, among them IC1 MPX5050DP, IC2 MPX5050DP, J1 Conn_01x04, J2 Conn_01x04, J3 Conn_01x06, J4 Micro match 6x2, J5 Conn_01x04, J6 Conn_01x06, J7 Conn_01x04, J8 Conn_01x06

Commit message: Fixes before ordering PCB
Signed-off-by: Jarosław Karwik <jaroslaw.karwik@gmail.com>
Parts:
- added U1: MPXH6115A, Biblioteki:MPXH6115AC6U, F.Cu at (116.2, 41.4)
- added U2: MPXH6115A, Biblioteki:MPXH6115AC6U, F.Cu at (139.1, 101.2)
Connections:
- IC1 pad 4: (no net) -> unconnected-(IC1-Pad4)
- IC1 pad 5: (no net) -> unconnected-(IC1-Pad5)
- IC1 pad 6: (no net) -> unconnected-(IC1-Pad6)
- IC2 pad 4: (no net) -> unconnected-(IC2-Pad4)
- IC2 pad 5: (no net) -> unconnected-(IC2-Pad5)
- IC2 pad 6: (no net) -> unconnected-(IC2-Pad6)
- J3 pad 2: (no net) -> unconnected-(J3-Pad2)
- J3 pad 3: (no net) -> unconnected-(J3-Pad3)
- J3 pad 6: (no net) -> unconnected-(J3-Pad6)
- J4 pad 1: (no net) -> unconnected-(J4-Pad1)
- J4 pad 10: (no net) -> unconnected-(J4-Pad10)
- J4 pad 13: (no net) -> unconnected-(J4-Pad13)
- J4 pad 14: (no net) -> unconnected-(J4-Pad14)
- J4 pad 15: (no net) -> unconnected-(J4-Pad15)
- J4 pad 16: (no net) -> unconnected-(J4-Pad16)
- J4 pad 17: (no net) -> unconnected-(J4-Pad17)
- J4 pad 18: (no net) -> unconnected-(J4-Pad18)
- J4 pad 2: (no net) -> unconnected-(J4-Pad2)
- J4 pad 23: (no net) -> unconnected-(J4-Pad23)
- J4 pad 24: (no net) -> unconnected-(J4-Pad24)
- J4 pad 25: (no net) -> unconnected-(J4-Pad25)
- J4 pad 26: (no net) -> unconnected-(J4-Pad26)
- J4 pad 27: (no net) -> unconnected-(J4-Pad27)
- J4 pad 28: (no net) -> unconnected-(J4-Pad28)
- J4 pad 9: (no net) -> unconnected-(J4-Pad9)
- J6 pad 2: (no net) -> unconnected-(J6-Pad2)
- J6 pad 3: (no net) -> unconnected-(J6-Pad3)
- J6 pad 6: (no net) -> unconnected-(J6-Pad6)
- J8 pad 2: (no net) -> unconnected-(J8-Pad2)
- J8 pad 3: (no net) -> unconnected-(J8-Pad3)
- J8 pad 6: (no net) -> unconnected-(J8-Pad6)
- SS1 pad 17: (no net) -> unconnected-(SS1-Pad17)
- SS1 pad 18: (no net) -> unconnected-(SS1-Pad18)
- SS2 pad 17: (no net) -> unconnected-(SS2-Pad17)
- SS2 pad 18: (no net) -> unconnected-(SS2-Pad18)
- SS3 pad 17: (no net) -> unconnected-(SS3-Pad17)
- SS3 pad 18: (no net) -> unconnected-(SS3-Pad18)
Routing:
- net +5V: track 170.4 -> 195.7 mm, vias 0 -> 1
- net Net-(IC2-Pad1): track 3.18 -> 12.5 mm, vias 0 -> 1
- net Net-(IC1-Pad1): track 26.3 -> 31.6 mm
- net GND: track 42.8 -> 46.3 mm, vias 31 -> 33
