File: hardware/10_shield_chm36VA/UniPrinterBase.kicad_sch (KiCad schematic)
At the start: 8 parts, among them J29 Conn_02x20_Odd_Even, J30 Conn_02x20_Odd_Even, J31 Conn_02x20_Odd_Even, J32 Conn_02x10_Odd_Even

Commit message: Fixes in PCB
Parts:
- J29, J30, J31, J32: footprint Connector_PinSocket_2.54mm:PinSocket_2x10_P2.54mm_Vertical_SMD -> Connector_PinHeader_2.54mm:PinHeader_2x10_P2.54mm_Vertical
Changed lines of the file:
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@@
       (effects (font (size 1.27 1.27)) hide)
     )
-    (property "Footprint" "Connector_PinSocket_2.54mm:PinSocket_2x10_P2.54mm_Vertical_SMD" (id 2) (at 90.17 142.24 0)
+    (property "Footprint" "Connector_PinHeader_2.54mm:PinHeader_2x10_P2.54mm_Vertical" (id 2) (at 90.17 142.24 0)
       (effects (font (size 1.27 1.27)) hide)
     )
@@
       (effects (font (size 1.27 1.27)) hide)
     )
-    (property "Footprint" "Connector_PinSocket_2.54mm:PinSocket_2x10_P2.54mm_Vertical_SMD" (id 2) (at 92.71 80.01 0)
+    (property "Footprint" "Connector_PinHeader_2.54mm:PinHeader_2x10_P2.54mm_Vertical" (id 2) (at 92.71 80.01 0)
       (effects (font (size 1.27 1.27)) hide)
     )
@@
       (effects (font (size 1.27 1.27)) hide)
     )
-    (property "Footprint" "Connector_PinSocket_2.54mm:PinSocket_2x10_P2.54mm_Vertical_SMD" (id 2) (at 92.71 111.76 0)
+    (property "Footprint" "Connector_PinHeader_2.54mm:PinHeader_2x10_P2.54mm_Vertical" (id 2) (at 92.71 111.76 0)
       (effects (font (size 1.27 1.27)) hide)
     )
@@
       (effects (font (size 1.27 1.27)) hide)
     )
-    (property "Footprint" "Connector_PinSocket_2.54mm:PinSocket_2x10_P2.54mm_Vertical_SMD" (id 2) (at 92.71 48.26 0)
+    (property "Footprint" "Connector_PinHeader_2.54mm:PinHeader_2x10_P2.54mm_Vertical" (id 2) (at 92.71 48.26 0)
       (effects (font (size 1.27 1.27)) hide)
     )

Commit message: Prepared for first prototype
Signed-off-by: Jarosław Karwik <jaroslaw.karwik@gmail.com>
Connections:
- net +3V3: now also J32.1 (Pin_1), J32.3 (Pin_3); no longer J32.2 (Pin_2), J32.4 (Pin_4)
- net +5V: now also J32.2 (Pin_2), J32.4 (Pin_4); no longer J32.1 (Pin_1), J32.3 (Pin_3)
- net ADC.CH1: now also J31.14 (Pin_14); no longer J31.13 (Pin_13)
- net ADC.CH2: now also J31.16 (Pin_16); no longer J31.15 (Pin_15)
- net DAC: now also J31.12 (Pin_12); no longer J31.11 (Pin_11)
- net ENC1.CH1: now also J32.5 (Pin_5); no longer J32.6 (Pin_6)
- net ENC1.CH2: now also J32.7 (Pin_7); no longer J32.8 (Pin_8)
- net ENC2.CH1: now also J32.6 (Pin_6); no longer J32.5 (Pin_5)
- net ENC2.CH2: now also J32.8 (Pin_8); no longer J32.7 (Pin_7)
- net ENC3_CH1.OUT_CPU11_PWM: now also J32.10 (Pin_10); no longer J32.9 (Pin_9)
- net ENC3_CH2.OUT_CPU12_PWM: now also J32.12 (Pin_12); no longer J32.11 (Pin_11)
- net IN_CPU1: now also J32.16 (Pin_16); no longer J32.15 (Pin_15)
- net IN_CPU2: now also J32.18 (Pin_18); no longer J32.17 (Pin_17)
- net IN_CPU3: now also J32.20 (Pin_20); no longer J32.19 (Pin_19)
- net IO_CPU1: now also J32.9 (Pin_9); no longer J32.10 (Pin_10)
- net IO_CPU2: now also J32.11 (Pin_11); no longer J32.12 (Pin_12)
- net IO_CPU3: now also J32.13 (Pin_13); no longer J32.14 (Pin_14)
- net IO_CPU4: now also J32.15 (Pin_15); no longer J32.16 (Pin_16)
- net IO_CPU5: now also J32.17 (Pin_17); no longer J32.18 (Pin_18)
- net IO_CPU6: now also J32.19 (Pin_19); no longer J32.20 (Pin_20)
- net IO_CPU7: now also J32.14 (Pin_14); no longer J32.13 (Pin_13)
- net IO_CPU8: now also J31.17 (Pin_17); no longer J31.18 (Pin_18)
- net IO_CPU9: now also J31.19 (Pin_19); no longer J31.20 (Pin_20)
- net LED: now also J31.10 (Pin_10); no longer J31.9 (Pin_9)
- net OUT_CPU10: now also J31.8 (Pin_8); no longer J31.7 (Pin_7)
- net OUT_CPU1_PWM: now also J30.10 (Pin_10); no longer J30.9 (Pin_9)
- net OUT_CPU2_PWM: now also J30.12 (Pin_12); no longer J30.11 (Pin_11)
- net OUT_CPU3_PWM: now also J30.14 (Pin_14); no longer J30.13 (Pin_13)
- net OUT_CPU4_PWM: now also J30.16 (Pin_16); no longer J30.15 (Pin_15)
- net OUT_CPU5: now also J30.18 (Pin_18); no longer J30.17 (Pin_17)
- net OUT_CPU6: now also J30.20 (Pin_20); no longer J30.19 (Pin_19)
- net OUT_CPU7: now also J31.2 (Pin_2); no longer J31.1 (Pin_1)
- net OUT_CPU8: now also J31.4 (Pin_4); no longer J31.3 (Pin_3)
- net OUT_CPU9: now also J31.6 (Pin_6); no longer J31.5 (Pin_5)
- net OUT_DIR1: now also J30.11 (Pin_11); no longer J30.12 (Pin_12)
- net OUT_DIR2: now also J30.15 (Pin_15); no longer J30.16 (Pin_16)
- net OUT_DIR3: now also J30.19 (Pin_19); no longer J30.20 (Pin_20)
- net OUT_DIR4: now also J31.3 (Pin_3); no longer J31.4 (Pin_4)
- net OUT_DIR5: now also J31.7 (Pin_7); no longer J31.8 (Pin_8)
- net OUT_DIR6: now also J31.11 (Pin_11); no longer J31.12 (Pin_12)
- net OUT_DIR7: now also J31.15 (Pin_15); no longer J31.16 (Pin_16)
- net OUT_STEP1: now also J30.9 (Pin_9); no longer J30.10 (Pin_10)
- net OUT_STEP2: now also J30.13 (Pin_13); no longer J30.14 (Pin_14)
- net OUT_STEP3: now also J30.17 (Pin_17); no longer J30.18 (Pin_18)
- net OUT_STEP4: now also J31.1 (Pin_1); no longer J31.2 (Pin_2)
- net OUT_STEP5: now also J31.5 (Pin_5); no longer J31.6 (Pin_6)
- net OUT_STEP6: now also J31.9 (Pin_9); no longer J31.10 (Pin_10)
- net OUT_STEP7: now also J31.13 (Pin_13); no longer J31.14 (Pin_14)
- net U6_485_A: now also J31.18 (Pin_18); no longer J31.17 (Pin_17)
- net U6_485_B: now also J31.20 (Pin_20); no longer J31.19 (Pin_19)
Changed lines of the file:
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@@
   (junction (at 97.79 101.6) (diameter 0) (color 0 0 0 0)
   )
+  (junction (at 85.09 132.08) (diameter 0) (color 0 0 0 0)
+  )
   (junction (at 85.09 43.18) (diameter 0) (color 0 0 0 0)
   )
@@
   )
   (junction (at 85.09 38.1) (diameter 0) (color 0 0 0 0)
-  )
-  (junction (at 85.09 132.08) (diameter 0) (color 0 0 0 0)
   )
   (junction (at 97.79 43.18) (diameter 0) (color 0 0 0 0)
@@
     (pin "1")
   )
-  (symbol (lib_id "Connector_Generic:Conn_02x10_Odd_Even") (at 92.71 80.01 0) (mirror y) (unit 1)
+  (symbol (lib_id "Connector_Generic:Conn_02x10_Odd_Even") (at 90.17 80.01 0) (unit 1)
     (in_bom yes) (on_board yes)
-    (property "Reference" "J31" (id 0) (at 92.71 67.31 0))
+    (property "Reference" "J31" (id 0) (at 90.17 67.31 0))
     (property "Value" "Conn_02x20_Odd_Even" (id 1) (at 91.44 54.102 0)
       (effects (font (size 1.27 1.27)) hide)
     )
-    (property "Footprint" "Connector_PinHeader_2.54mm:PinHeader_2x10_P2.54mm_Vertical" (id 2) (at 92.71 80.01 0)
-      (effects (font (size 1.27 1.27)) hide)
-    )
-    (property "Datasheet" "~" (id 3) (at 92.71 80.01 0)
+    (property "Footprint" "Connector_PinHeader_2.54mm:PinHeader_2x10_P2.54mm_Vertical" (id 2) (at 90.17 80.01 0)
+      (effects (font (size 1.27 1.27)) hide)
+    )
+    (property "Datasheet" "~" (id 3) (at 90.17 80.01 0)
       (effects (font (size 1.27 1.27)) hide)
     )
@@
     (pin "1")
   )
-  (symbol (lib_id "Connector_Generic:Conn_02x10_Odd_Even") (at 92.71 111.76 0) (mirror y) (unit 1)
+  (symbol (lib_id "Connector_Generic:Conn_02x10_Odd_Even") (at 90.17 111.76 0) (unit 1)
     (in_bom yes) (on_board yes) (fields_autoplaced)
     (property "Reference" "J32" (id 0) (at 91.44 97.79 0))
@@
       (effects (font (size 1.27 1.27)) hide)
     )
-    (property "Footprint" "Connector_PinHeader_2.54mm:PinHeader_2x10_P2.54mm_Vertical" (id 2) (at 92.71 111.76 0)
-      (effects (font (size 1.27 1.27)) hide)
-    )
-    (property "Datasheet" "~" (id 3) (at 92.71 111.76 0)
+    (property "Footprint" "Connector_PinHeader_2.54mm:PinHeader_2x10_P2.54mm_Vertical" (id 2) (at 90.17 111.76 0)
+      (effects (font (size 1.27 1.27)) hide)
+    )
+    (property "Datasheet" "~" (id 3) (at 90.17 111.76 0)
       (effects (font (size 1.27 1.27)) hide)
     )
@@
     (pin "9")
   )
-  (symbol (lib_id "Connector_Generic:Conn_02x10_Odd_Even") (at 92.71 48.26 0) (mirror y) (unit 1)
+  (symbol (lib_id "Connector_Generic:Conn_02x10_Odd_Even") (at 90.17 48.26 0) (unit 1)
     (in_bom yes) (on_board yes) (fields_autoplaced)
     (property "Reference" "J30" (id 0) (at 91.44 34.29 0))
@@
       (effects (font (size 1.27 1.27)) hide)
     )
-    (property "Footprint" "Connector_PinHeader_2.54mm:PinHeader_2x10_P2.54mm_Vertical" (id 2) (at 92.71 48.26 0)
-      (effects (font (size 1.27 1.27)) hide)
-    )
-    (property "Datasheet" "~" (id 3) (at 92.71 48.26 0)
-      (effects (font (size 1.27 1.27)) hide)
-    )
+    (property "Footprint" "Connector_PinHeader_2.54mm:PinHeader_2x10_P2.54mm_Vertical" (id 2) (at 90.17 48.26 0)
+      (effects (font (size 1.27 1.27)) hide)
+    )
+    (property "Datasheet" "~" (id 3) (at 90.17 48.26 0)
+      (effects (font (size 1.27 1.27)) hide)
+    )
