File: hardware/11_shield_CHM36VA/controller.kicad_sch (KiCad schematic)
At the start: 44 parts, among them Q1 IRLL2705PBF, Q10 IRLL2705PBF, Q2 IRLL2705PBF, Q3 IRLL2705PBF, Q4 IRLL2705PBF, Q5 IRLL2705PBF, Q6 BSS138BKS, Q7 IRLL2705PBF, Q8 IRLL2705PBF, Q9 BSS138BKS, U1 LM217_TO-252, U2 AM26LS32ACD, U3 CNY17-1

Commit message: 1.New shield version 1.1
Parts:
- added D8, D9: SK56, Diode_SMD:D_SMB, symbol Device:D_Schottky
- renumbered D8 to D10, Q9 to Q7, Q7 to Q8, Q8 to Q9
Connections:
- net +24V: now also D10.1 (K), D3.1 (K), D4.1 (K), D5.1 (K), D6.1 (K), D7.1 (K), D8.1 (K), D9.1 (K)
- net GND: no longer D10.2 (A), D3.2 (A), D4.2 (A), D5.2 (A), D6.2 (A), D7.2 (A)
- net OUT_LED_DN: now also D9.2 (A)
- net OUT_LED_UP: now also D8.2 (A)
- net OUT_LZ: now also D3.2 (A); no longer D3.1 (K)
- net OUT_N1_VALVE: now also D6.2 (A); no longer D6.1 (K)
- net OUT_N2_VALVE: now also D10.2 (A); no longer D10.1 (K)
- net OUT_UNUSED: now also D7.2 (A); no longer D7.1 (K)
- net PUMP_PRESS: now also D5.2 (A); no longer D5.1 (K)
- net PUMP_VACUUM: now also D4.2 (A); no longer D4.1 (K)
Other:
- moved on the sheet: D10, D3, D4, D5, D6, D7, Q7B
