File: hardware/11_shield_CHM36VA/shield_chm36VA.kicad_pcb (KiCad board)
At the start: 2 copper layers, 199.6 x 100 mm, 71 parts, among them J10 Conn_01x06_Male, J11 Conn_01x10_Male, J12 Conn_01x10_Male, J14 Conn_01x09_Male, J15 Conn_01x02_Male, J17 Conn_01x06_Male, J20 Conn_01x09_Male, J21 Conn_01x02_Male, J23 Conn_01x10_Male, J25 Conn_01x02_Male, J26 Conn_01x10_Male, J27 Conn_01x10_Male, J28 Conn_02x05_Odd_Even, J29 Conn_02x05_Odd_Even, J3 Conn_01x06_Male, J30 Conn_02x20_Odd_Even, J31 Conn_02x20_Odd_Even, J32 Conn_02x10_Odd_Even, J33 Conn_02x20_Odd_Even, J4 Conn_01x04_Male, J5 Conn_01x10_Male, J7 Conn_01x04_Male, J8 Conn_02x05_Odd_Even, Q1 IRLL2705PBF, Q10 IRLL2705PBF, Q2 IRLL2705PBF, Q3 IRLL2705PBF, Q4 IRLL2705PBF, Q5 IRLL2705PBF, Q6 BSS138BKS, Q7 IRLL2705PBF, Q8 IRLL2705PBF, Q9 BSS138BKS, U1 LM217_TO-252, U2 AM26LS32ACD, U3 CNY17-1

Commit message: 1.New shield version 1.1
Parts:
- added D8: SK56, Diode_SMD:D_SMB, F.Cu at (62.5, 67.1)
- added D9: SK56, Diode_SMD:D_SMB, F.Cu at (69.5, 67.1)
- moved R8 4.02 mm to (92.3, 90.6)
- moved D6 3.50 mm to (77.0, 67.1), turned to 90 degrees
- moved D10 3.50 mm to (84.5, 67.5), turned to 90 degrees
- moved D7 2.53 mm to (91.0, 67.1), turned to 90 degrees
- moved D3 0.40 mm to (96.0, 67.1), turned to 90 degrees
- turned D4 to 180 degrees
- turned D5 to 180 degrees
- renumbered D8 to D10, Q9 to Q7, Q7 to Q8, Q8 to Q9
Connections:
- D10 pad 1: /controller/OUT_N2_VALVE -> +24V
- D10 pad 2: GND -> /controller/OUT_N2_VALVE
- D3 pad 1: /controller/OUT_LZ -> +24V
- D3 pad 2: GND -> /controller/OUT_LZ
- D4 pad 1: /controller/PUMP_VACUUM -> +24V
- D4 pad 2: GND -> /controller/PUMP_VACUUM
- D5 pad 1: /controller/PUMP_PRESS -> +24V
- D5 pad 2: GND -> /controller/PUMP_PRESS
- D6 pad 1: /controller/OUT_N1_VALVE -> +24V
- D6 pad 2: GND -> /controller/OUT_N1_VALVE
- D7 pad 1: /controller/OUT_UNUSED -> +24V
- D7 pad 2: GND -> /controller/OUT_UNUSED
Routing:
- net /controller/ENC_Y_B+: track 265.6 -> 20.9 mm, vias 5 -> 0
- net +5V: track 370.8 -> 538.6 mm, vias 3 -> 9
- net +24V: track 169.5 -> 300.3 mm, vias 0 -> 15
- net /controller/UniPrinterBase/ENC1.CH1: track 0.00 -> 123.7 mm, vias 0 -> 2
- net /controller/UniPrinterBase/ENC1.CH2: track 0.00 -> 118.4 mm, vias 0 -> 2
- net /controller/SPARE_OUT11: track 0.00 -> 115.6 mm, vias 0 -> 2
- net /controller/SPARE_OUT10: track 0.00 -> 115.0 mm, vias 0 -> 2
- net /controller/UniPrinterBase/OUT_CPU8: track 0.00 -> 97.9 mm, vias 0 -> 2
- net /controller/SPARE_STEP_D: track 0.00 -> 89.6 mm, vias 0 -> 2
- net /controller/SPARE_DIR_D: track 0.00 -> 84.1 mm, vias 0 -> 3
- net /controller/SPARE_IO3: track 0.00 -> 73.8 mm, vias 0 -> 1
- net /controller/SPARE_IO4: track 0.00 -> 72.5 mm, vias 0 -> 1
- net /controller/SPARE_IO5: track 0.00 -> 72.3 mm, vias 0 -> 1
- net /controller/ENC_X_A+: track 0.00 -> 58.9 mm, vias 0 -> 1
- net /controller/ENC_X_A-: track 112.6 -> 57.6 mm, vias 2 -> 1
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- removed copper zone on F.Cu, net +5V
