File: hardware/00_Uni_Printer/Power_supply.kicad_sch (KiCad schematic)
At the start: 11 parts, among them IC1 MAX17503ATP+, IC4 TLV1117-33

Commit message: New idea - mix project will take over
Signed-off-by: Jaroslaw Karwik <jaroslaw.karwik@gmail.com>
Parts:
- renumbered C40 to C1, C1 to C2, C42 to C3, C41 to C4, C43 to C5, C44 to C6, IC4 to IC2, L2 to L1, R52 to R1, R53 to R2
