File: hardware/00_Uni_Printer/Uni_Printer.kicad_sch (KiCad schematic)
At the start: 65 parts, among them J1 Conn_01x04_Male, J2 FIDUCIAL, J4 Conn_01x06, J5 Conn_02x10_Odd_Even, J6 Conn_02x10_Odd_Even, J6 FIDUCIAL, J7 Conn_02x10_Odd_Even, J8 Conn_02x10_Odd_Even, U2 74AHC04, U3 74AHC04, U6 LM2904

Commit message: New idea - mix project will take over
Signed-off-by: Jaroslaw Karwik <jaroslaw.karwik@gmail.com>
Parts:
- renumbered D1 to D10, D1 to D11, D1 to D12, D1 to D13, D1 to D14, D1 to D15, D3 to D16, D1 to D2, D1 to D3, D2 to D5, D1 to D6, D1 to D7, D1 to D8, D1 to D9, J6 to J3, MK6 to MK4, R4 to R13, R4 to R14, R4 to R17, R4 to R18, R4 to R19, RN6 to RN10, RN6 to RN11, RN6 to RN12, RN1 to RN13, RN6 to RN14, RN6 to RN15, RN6 to RN16, RN6 to RN17, RN6 to RN18, RN6 to RN19, RN6 to RN2, RN6 to RN20, RN6 to RN23, RN6 to RN24, RN6 to RN25, RN6 to RN27, RN6 to RN28, RN6 to RN3, RN6 to RN4, RN6 to RN5, RN6 to RN7, RN6 to RN8, RN6 to RN9
