File: hardware/00_Uni_Printer/ethernet.kicad_sch (KiCad schematic)
At the start: 27 parts, among them IC5 LAN8742A, J11 LMJ1998824110DL1T39J, Y2 ABM7-25.000MHZ-D2Y-T

Commit message: New idea - mix project will take over
Signed-off-by: Jaroslaw Karwik <jaroslaw.karwik@gmail.com>
Parts:
- renumbered C4 to C22, C5 to C23, C6 to C24, C7 to C25, C9 to C26, C21 to C27, C33 to C28, C35 to C29, C36 to C30, C37 to C31, IC5 to IC4, J11 to J9, L1 to L2, R46 to R10, R47 to R11, R48 to R12, R38 to R20, R38 to R21, R38 to R22, R1 to R6, R2 to R7, R38 to R8, R45 to R9, RN10 to RN21
