File: hardware/00_Uni_Printer/processor.kicad_sch (KiCad schematic)
At the start: 22 parts, among them IC2 MT25QL256ABA1EW7-0SIT_TR, U1 STM32H743VIT6, Y1 ABM7-25.000MHZ-D2Y-T

Commit message: New idea - mix project will take over
Signed-off-by: Jaroslaw Karwik <jaroslaw.karwik@gmail.com>
Parts:
- renumbered C14 to C10, C2 to C12, C15 to C13, C13 to C14, C17 to C15, C20 to C16, C22 to C17, C23 to C20, C24 to C21, C16 to C7, C10 to C8, C12 to C9, IC2 to IC3, R4 to R3, R5 to R4, R3 to R5
