File: hardware/12_mixture/UniMixFeeders/UniMixFeeders.kicad_pcb (KiCad board)
At the start: 2 copper layers, 365 x 32 mm, 124 parts, among them IC1 AP7375-33W5-7, IC2 LPC11C22FBD48_301,, J1 Conn_01x04_Male, J10 Conn_01x04_Pin, J11 Conn_01x04_Pin, J12 Conn_01x04_Pin, J13 Conn_01x04_Pin, J14 Conn_01x10_Pin, J15 Conn_01x04_Pin, J16 Conn_01x04_Pin, J17 Conn_01x04_Pin, J18 Conn_01x04_Pin, J19 Conn_01x04_Pin, J2 Conn_01x04_Male, J20 Conn_01x04_Pin, J21 Conn_01x04_Pin, J22 Conn_01x04_Pin, J23 Conn_01x04_Pin, J24 Conn_01x04_Pin, J25 Conn_01x04_Pin, J26 Conn_01x04_Pin, J27 Conn_01x04_Pin, J28 Conn_01x04_Pin, J29 Conn_01x04_Pin, J3 Conn_01x04_Pin, J30 Conn_01x04_Pin, J31 Conn_01x04_Pin, J32 Conn_01x04_Pin, J4 Conn_01x04_Pin, J6 Conn_01x04_Pin, J7 Conn_01x04_Pin, J8 Conn_01x04_Pin, J9 Conn_01x04_Pin, Y1 ABM7-20.000MHZ-D2Y-T

Commit message: CAN FD head added
Parts:
- removed C20, C32, C34, C35, C36: 10uF, Capacitor_SMD:C_1206_3216Metric
- removed D2: BAV99S, Package_TO_SOT_SMD:SOT-363_SC-70-6
- removed J14: Conn_01x10_Pin, Connector_PinHeader_2.54mm:PinHeader_1x12_P2.54mm_Vertical
- removed J28, J29, J30, J31, J32: Conn_01x04_Pin, Connector_PinHeader_2.54mm:PinHeader_1x04_P2.54mm_Vertical
- removed JP3, JP6: Jumper_2_Open, Jumper:SolderJumper-2_P1.3mm_Open_RoundedPad1.0x1.5mm
- removed JP4, JP5: Jumper_2_Open, Jumper:SolderJumper-2_P1.3mm_Bridged_RoundedPad1.0x1.5mm
- removed R24, R25, R26, R27, R31, R32: 1k, Resistor_SMD:R_0603_1608Metric
- added F2: PTSLR12106V175, Fuse:Fuse_1210_3225Metric, F.Cu at (405.6, 126.1)
- added H3: MountingHole, MountingHole:MountingHole_3.2mm_M3, F.Cu at (393.1, 131.5)
- added J5: Conn_01x04_Pin, Connector_PinHeader_2.54mm:PinHeader_1x04_P2.54mm_Vertical, B.Cu at (402.2, 134.5)
- C1, C4, C5, IC1, JP1, JP2: moved to B.Cu
- H1, H11, H12, H14, H2, H4, H5, H7, H8, H9: footprint MountingHole:MountingHole_3.2mm_M3_DIN965_Pad -> MountingHole:MountingHole_3.2mm_M3
- J16: value Conn_01x04_Pin -> Conn_01x06_Pin; footprint Connector_PinHeader_2.54mm:PinHeader_1x04_P2.54mm_Vertical -> Connector_PinHeader_2.54mm:PinHeader_1x06_P2.54mm_Vertical; moved to F.Cu
- J27: value Conn_01x04_Pin -> Conn_01x06_Pin; footprint Connector_PinHeader_2.54mm:PinHeader_1x04_P2.54mm_Vertical -> Connector_PinHeader_2.54mm:PinHeader_2x03_P2.54mm_Vertical; moved to F.Cu
- moved J16 265.6 mm to (41.4, 138.3), turned to 90 degrees
- moved J27 167.0 mm to (153.1, 129.5), turned to 90 degrees
- moved C26 111.7 mm to (362.5, 127.9), turned to 90 degrees
- moved C28 103.9 mm to (380.7, 128.0), turned to 90 degrees
- moved C4 98.9 mm to (216.2, 125.1), turned to 0 degrees
- moved C1 98.9 mm to (216.2, 126.9), turned to 0 degrees
- moved C30 96.2 mm to (399.0, 128.0), turned to 90 degrees
- moved R10 92.6 mm to (399.5, 133.0), turned to -90 degrees
- moved IC1 91.3 mm to (212.3, 125.9), turned to 180 degrees
- moved R9 90.0 mm to (381.2, 133.1)
- moved J15 90.0 mm to (384.0, 134.5)
- moved R4 84.9 mm to (363.1, 133.0)
- moved J26 84.8 mm to (365.8, 134.5)
- moved C5 84.1 mm to (208.4, 125.3)
- moved R3 80.5 mm to (344.8, 133.2), turned to -90 degrees
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Connections:
- J1 pad 2: /COM_H -> /CANH
- J1 pad 3: /COM_L -> /CANL
- J16 pad 1: unconnected-(J16-Pin_1-Pad1) -> GND
- J16 pad 2: /S22 -> unconnected-(J16-Pin_2-Pad2)
- J16 pad 3: +5V -> unconnected-(J16-Pin_3-Pad3)
- J16 pad 4: GND -> Net-(J16-Pin_4)
- J2 pad 1: Net-(J1-Pin_1) -> Net-(J2-Pin_1)
- J2 pad 2: /COM_H -> /CANH
- J2 pad 3: /COM_L -> /CANL
- J27 pad 1: unconnected-(J27-Pin_1-Pad1) -> /BOOT
- J27 pad 2: /S23 -> +3.3V
- J27 pad 3: +5V -> /RESET
- J27 pad 4: GND -> /SWDIO
- JP1 pad 1: /P02 -> /P11
- JP2 pad 1: /P18 -> /P10
- R10 pad 2: /P06 -> /P18
- R11 pad 2: /P211 -> /P05
- R12 pad 2: /P110 -> /P04
- R16 pad 2: /P12 -> /P07
- R17 pad 2: /P09 -> /P03
- R18 pad 2: /P08 -> /P21
- R23 pad 2: /P11 -> /P210
- R28 pad 2: Net-(J14-Pin_11) -> Net-(J16-Pin_5)
- R29 pad 1: Net-(J14-Pin_10) -> Net-(J16-Pin_4)
- R3 pad 2: /P22 -> /P02
- R4 pad 2: /P210 -> /P28
- R5 pad 2: /P10 -> /P22
- R6 pad 2: /P011 -> /P08
- R9 pad 2: /P07 -> /P27
Routing:
- net +5V: track 746.2 -> 101.9 mm, vias 2 -> 14
- net GND: track 519.4 -> 107.3 mm, vias 43 -> 20
- net /CANH: track 26.1 -> 429.2 mm
- net /CANL: track 30.6 -> 432.0 mm
- net /COM_H: track 365.1 -> 0.00 mm, vias 4 -> 0
- net /COM_L: track 363.0 -> 0.00 mm, vias 2 -> 0
- net Net-(J1-Pin_1): track 357.3 -> 7.12 mm
- net /P18: track 21.1 -> 210.9 mm
- net /P06: track 135.2 -> 0.00 mm
- net /P02: track 20.6 -> 155.4 mm
- net /P07: track 117.7 -> 10.5 mm
- net /P05: track 151.8 -> 79.6 mm
- net /P210: track 103.8 -> 35.0 mm
- net /P04: track 166.0 -> 97.9 mm
- net /P09: track 65.2 -> 0.00 mm
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- added copper zone on In2.Cu, net +3.3V
- added copper zone on B.Cu, net +5V
- added copper zone on In2.Cu, net +5V
- added copper zone on In1.Cu, net GND
- removed copper zone on B.Cu, net +3.3V
- removed copper zone on B.Cu, net GND
Other:
- board size 365 x 32 mm -> 409.6 x 20 mm
- copper layers 2 -> 4
- board text added: "+3V3"
- board text added: "BOOT"
- board text added: "GND"
- board text added: "RESET"
- board text added: "SWCLK"
- board text added: "SWDIO"
- board text added: "UniMixFeeders v1.1 jaroslaw.karwik@gmail.com github.com/jarekkt/UniController"
- board text removed: "23"
- board text removed: "24"
- board text removed: "25"
- board text removed: "26"
- board text removed: "27"
- board text removed: "28"
- board text removed: "UniMixFeeders v1.0 jaroslaw.karwik@gmail.com github.com/jarekkt/UniController"
