File: hardware/12_mixture/UniMixFeeders/UniMixFeeders.kicad_sch (KiCad schematic)
At the start: 124 parts, among them IC1 AP7375-33W5-7, IC2 LPC11C22FBD48_301,, J1 Conn_01x04_Male, J10 Conn_01x04_Pin, J11 Conn_01x04_Pin, J12 Conn_01x04_Pin, J13 Conn_01x04_Pin, J14 Conn_01x10_Pin, J15 Conn_01x04_Pin, J16 Conn_01x04_Pin, J17 Conn_01x04_Pin, J18 Conn_01x04_Pin, J19 Conn_01x04_Pin, J2 Conn_01x04_Male, J20 Conn_01x04_Pin, J21 Conn_01x04_Pin, J22 Conn_01x04_Pin, J23 Conn_01x04_Pin, J24 Conn_01x04_Pin, J25 Conn_01x04_Pin, J26 Conn_01x04_Pin, J27 Conn_01x04_Pin, J28 Conn_01x04_Pin, J29 Conn_01x04_Pin, J3 Conn_01x04_Pin, J30 Conn_01x04_Pin, J31 Conn_01x04_Pin, J32 Conn_01x04_Pin, J4 Conn_01x04_Pin, J6 Conn_01x04_Pin, J7 Conn_01x04_Pin, J8 Conn_01x04_Pin, J9 Conn_01x04_Pin, Y1 ABM7-20.000MHZ-D2Y-T

Commit message: CAN FD head added
Parts:
- removed C20, C32, C34, C35, C36: 10uF, Capacitor_SMD:C_1206_3216Metric, symbol Device:C
- removed D2: BAV99S, Package_TO_SOT_SMD:SOT-363_SC-70-6, symbol Diode:BAV99S
- removed J14: Conn_01x10_Pin, Connector_PinHeader_2.54mm:PinHeader_1x12_P2.54mm_Vertical, symbol Connector:Conn_01x12_Pin
- removed J16, J27, J28, J29, J30, J31, J32: Conn_01x04_Pin, Connector_PinHeader_2.54mm:PinHeader_1x04_P2.54mm_Vertical, symbol Connector:Conn_01x04_Pin
- removed JP3, JP6: Jumper_2_Open, Jumper:SolderJumper-2_P1.3mm_Open_RoundedPad1.0x1.5mm, symbol Jumper:Jumper_2_Open
- removed JP4, JP5: Jumper_2_Open, Jumper:SolderJumper-2_P1.3mm_Bridged_RoundedPad1.0x1.5mm, symbol Jumper:Jumper_2_Bridged
- removed R24, R25, R26, R27, R31, R32: 1k, Resistor_SMD:R_0603_1608Metric, symbol Device:R
- added F2: PTSLR12106V175, Fuse:Fuse_1210_3225Metric, symbol Device:Polyfuse
- added H3: MountingHole, MountingHole:MountingHole_3.2mm_M3, symbol Mechanical:MountingHole
- added J16: Conn_01x06_Pin, Connector_PinHeader_2.54mm:PinHeader_1x06_P2.54mm_Vertical, symbol Connector:Conn_01x06_Pin
- added J27: Conn_01x06_Pin, Connector_PinHeader_2.54mm:PinHeader_2x03_P2.54mm_Vertical, symbol Connector:Conn_01x06_Pin
- added J5: Conn_01x04_Pin, Connector_PinHeader_2.54mm:PinHeader_1x04_P2.54mm_Vertical, symbol Connector:Conn_01x04_Pin
- H1, H11, H12, H14, H2, H4, H5, H7, H8, H9: footprint MountingHole:MountingHole_3.2mm_M3_DIN965_Pad -> MountingHole:MountingHole_3.2mm_M3
Connections:
- net COM_H is gone; now on net CANH: J1.2 (Pin_2), J2.2 (Pin_2)
- net COM_L is gone; now on net CANL: J1.3 (Pin_3), J2.3 (Pin_3)
- net +3.3V: now also J27.2 (Pin_2)
- net +5V: now also F2.1, J5.3 (Pin_3)
- net BOOT: now also J27.1 (Pin_1)
- net GND: now also J16.1 (Pin_1), J27.6 (Pin_6), J5.4 (Pin_4)
- net P011: no longer R6.2
- net P02: now also R3.2; no longer JP1.1 (A)
- net P03: now also R17.2
- net P04: now also R12.2
- net P05: now also R11.2
- net P06: no longer R10.2
- net P07: now also R16.2; no longer R9.2
- net P08: now also R6.2; no longer R18.2
- net P09: no longer R17.2
- net P10: now also JP2.1 (A); no longer R5.2
- net P11: now also JP1.1 (A); no longer R23.2
- net P110: no longer R12.2
- net P12: no longer R16.2
- net P18: now also R10.2; no longer JP2.1 (A)
- net P21: now also R18.2
- net P210: now also R23.2; no longer R4.2
- net P211: no longer R11.2
- net P22: now also R5.2; no longer R3.2
- net P27: now also R9.2
- net P28: now also R4.2
- net RESET: now also J27.3 (Pin_3)
- net S22: now also J5.2 (Pin_2)
- net SWCLK: now also J27.5 (Pin_5)
- net SWDIO: now also J27.4 (Pin_4)
- net at R29.1: now also J16.4 (Pin_4)
- net at R28.2: now also J16.5 (Pin_5)
- net at F1.2, J1.1 (Pin_1): no longer J2.1 (Pin_1)
- new net: F2.2, J2.1 (Pin_1)
- no-connect marks 31 -> 25
Other:
- moved on the sheet: F1, R28, R29
